File: file5A05C1E8.sch (KiCad schematic (older format))
At the start: 9 parts

Commit message: updated to new kicad format
Parts:
- C? (x3): symbol C_Small -> Device:C_Small
Changed lines of the file:
@@
 $EndComp
 $Comp
-L C_Small C?
+L Device:C_Small C?
 U 1 1 5A05C39F
 P 6100 2750
@@
 $EndComp
 $Comp
-L C_Small C?
+L Device:C_Small C?
 U 1 1 5A05C3E3
 P 6650 2750
@@
 $EndComp
 $Comp
-L C_Small C?
+L Device:C_Small C?
 U 1 1 5A05D8CA
 P 5350 2800
