File: file5A0600C5.sch (KiCad schematic (older format))
At the start: 6 parts

Commit message: updated to new kicad format
Parts:
- C? (x4): symbol C_Small -> Device:C_Small
Changed lines of the file:
@@
 $EndComp
 $Comp
-L C_Small C?
+L Device:C_Small C?
 U 1 1 5A0602B6
 P 4800 2350
@@
 $EndComp
 $Comp
-L C_Small C?
+L Device:C_Small C?
 U 1 1 5A0602BD
 P 5100 2700
@@
 $EndComp
 $Comp
-L C_Small C?
+L Device:C_Small C?
 U 1 1 5A0602D7
 P 4600 2650
@@
 $EndComp
 $Comp
-L C_Small C?
+L Device:C_Small C?
 U 1 1 5A0602DE
 P 4600 3300
