File: USB-DAC.kicad_pcb (KiCad board)
At the start: 2 copper layers, 138 parts, among them J1 USB_B, J3 BARREL_JACK, U1 S25FL116K0XNFA013, U10 L78L15_SO8, U11 L79L15_SO8, U12 TPS563209, U13 TPS563209, U14 AK4452, U15 NE5534, U16 NE5534, U17 DRV135, U18 DRV135, U19 TPA6120A2, U2 74LV14, U3 XHRA-2HPA, U4 NCP303LSN09T1G, U5 74LV74, U6 74LV157, U7 LM27313, U8 LM43601, U9 L78L05_SO8, Y1 24, Y2 24.576, Y3 22.5792

Commit message: Began PCB layout
Parts:
- removed C17, C18, C19: 18p, Capacitors_SMD:C_0805_HandSoldering
- removed C28: 120p, Capacitors_SMD:C_0805_HandSoldering
- removed C29, C30, C38: 4u7, Capacitors_SMD:C_0805_HandSoldering
- removed C32, C35, C36, C37: 10u, Capacitors_SMD:C_0805_HandSoldering
- removed D2: SK34ATR, Diodes_SMD:D_SMA_Handsoldering
- removed F1: 2A, Resistors_SMD:R_1812_HandSoldering
- removed L1: 10u, Inductors_SMD:L_7.3x7.3_H3.5
- removed L2: 56u, Inductors_SMD:L_12x12mm_h4.5mm
- removed R10, R4, R9: 220, Resistors_SMD:R_0805_HandSoldering
- removed R16: 187K, Resistors_SMD:R_0805_HandSoldering
- removed R17, R3, R7, R8: 1M, Resistors_SMD:R_0805_HandSoldering
- removed U2: 74LV14, Housings_SOIC:SOIC-14_3.9x8.7mm_Pitch1.27mm
- added J2: SPDIF OUT, dacparts:pjras1x1s_series, F.Cu at (137.2, 50.8)
- added J4: JACK_TRS_6PINS, Connectors:NMJ6HCD2, F.Cu at (148.6, 54.6)
- added J5: JACK_TRS_6PINS, Connectors:NMJ6HCD2, F.Cu at (168.9, 54.6)
- added J6: JACK_TRS_6PINS, Connectors:NMJ6HCD2, F.Cu at (185.1, 156.2)
- added RV1: P10K, dacparts:PTR90, F.Cu at (102.9, 154.9)
- C16, C5, C7: value 18p -> 100n
- C22: value 2u2 -> 22u
- C24: value 470n -> 22u
- C27: value 110p -> 100n
- C63, C64, C65, C66: value 0.1u -> 100n
- R1: value 10K -> 0
- R13: value 1K -> 0
- R14: value 60K4 -> 0
- R15: value 13K7 -> 0
- R36: value 50 -> 51
- U1: value S25FL116K0XNFA013 -> ISO7340FC; footprint Housings_SON:WSON-8_1EP_2x2mm_Pitch0.5mm -> Housings_SOIC:SOIC-16W_7.5x10.3mm_Pitch1.27mm
- U10: value L78L15_SO8 -> L79L12_SO8
- U11: value L79L15_SO8 -> AP1117-33; footprint Housings_SOIC:SOIC-8_3.9x4.9mm_Pitch1.27mm -> TO_SOT_Packages_SMD:SOT-223-3_TabPin2
- U5: value 74LV74 -> 74LVC1G79; footprint Housings_SOIC:SOIC-14_3.9x8.7mm_Pitch1.27mm -> TO_SOT_Packages_SMD:SOT-353_SC-70-5_Handsoldering
- U6: value 74LV157 -> TC7WH157; footprint Housings_SOIC:SOIC-16_3.9x9.9mm_Pitch1.27mm -> Housings_SSOP:SSOP-8_2.95x2.8mm_Pitch0.65mm
- U7: value LM27313 -> CHINADCDC; footprint TO_SOT_Packages_SMD:SOT-23-5_HandSoldering -> dacparts:chinadcdc
- U8: value LM43601 -> LM78L12_SO8; footprint Housings_SSOP:SSOP-16_4.4x5.2mm_Pitch0.65mm -> Housings_SOIC:SOIC-8_3.9x4.9mm_Pitch1.27mm
- Y1, Y2: footprint Crystals:Crystal_SMD_HC49-SD_HandSoldering -> Crystals:Crystal_SMD_3225-4pin_3.2x2.5mm
- Y3: footprint Crystals:Crystal_SMD_HC49-SD_HandSoldering -> Crystals:Crystal_SMD_2016-4pin_2.0x1.6mm
- moved R22 225.4 mm to (367.9, 53.4)
- moved R24 224.2 mm to (367.9, 58.9)
- moved R27 222.0 mm to (366.8, 64.4)
- moved R26 220.4 mm to (362.7, 53.4)
- moved R31 219.1 mm to (362.7, 58.9)
- moved R23 217.0 mm to (361.6, 64.4)
- moved C49 215.4 mm to (357.7, 53.5)
- moved R28 212.8 mm to (356.3, 59.0)
- moved R33 211.9 mm to (356.5, 64.5)
- moved R25 211.1 mm to (356.7, 70.0)
- moved C56 210.6 mm to (352.7, 53.5)
- moved C61 207.9 mm to (351.2, 59.0)
- moved R29 206.8 mm to (351.3, 64.5)
- moved R32 206.0 mm to (351.5, 70.0)
- moved C54 205.8 mm to (347.8, 53.5)
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Connections:
- C1 pad 1: +3V3 -> VCC
- C10 pad 2: GND -> GNDD
- C11 pad 2: GND -> GNDD
- C12 pad 2: GND -> GNDD
- C13 pad 2: GND -> GNDD
- C14 pad 2: GND -> GNDD
- C15 pad 2: GND -> GNDD
- C16 pad 1: Net-(C16-Pad1) -> +3V3
- C16 pad 2: GND -> GNDD
- C2 pad 2: GND -> GNDD
- C21 pad 1: GND -> GNDD
- C22 pad 2: /Power Supply/-18V -> GND
- C23 pad 1: +3V3 -> VCC
- C24 pad 1: Net-(C24-Pad1) -> GND
- C25 pad 1: +3V3 -> VCC
- C26 pad 1: +3V3 -> VCC
- C27 pad 1: /Power Supply/+18V -> +3.3VA
- C27 pad 2: Net-(C27-Pad2) -> GND
- C3 pad 2: GND -> GNDD
- C33 pad 1: /Power Supply/+18V -> Net-(C22-Pad1)
- C34 pad 2: /Power Supply/-18V -> Net-(C24-Pad2)
- C39 pad 1: +15V -> +12V
- C4 pad 2: GND -> GNDD
- C40 pad 2: -12VA -> -12V
- C42 pad 2: Net-(C42-Pad2) -> GNDD
- C43 pad 2: Net-(C42-Pad2) -> GNDD
- C44 pad 2: Net-(C42-Pad2) -> GNDD
- C46 pad 2: Net-(C46-Pad2) -> GNDD
- C47 pad 2: Net-(C46-Pad2) -> GNDD
- C48 pad 2: Net-(C46-Pad2) -> GNDD
- C49 pad 1: +3V3 -> +3.3VA
- C5 pad 1: Net-(C5-Pad1) -> +3V3
- C5 pad 2: GND -> GNDD
- C50 pad 1: +3V3 -> +3.3VA
- C51 pad 2: GND -> GNDD
- C52 pad 2: GND -> GNDD
- C53 pad 2: GND -> GNDD
- C54 pad 1: GND -> GNDD
- C6 pad 2: GND -> GNDD
- C7 pad 1: Net-(C7-Pad1) -> +3V3
- C7 pad 2: GND -> GNDD
- C8 pad 2: GND -> GNDD
- C9 pad 2: GND -> GNDD
- D1 pad 1: +3V3 -> VCC
- D1 pad 2: GND -> Net-(D1-Pad2)
- J1 pad 1: Net-(J1-Pad1) -> VBUS
- J1 pad 4: GND -> GNDD
- J1 pad 5: GND -> GNDD
- J3 pad 1: Net-(F1-Pad2) -> Net-(D1-Pad2)
- R1 pad 1: /USB/~CS -> Net-(R1-Pad1)
- R12 pad 1: GND -> GNDD
- R14 pad 1: /Power Supply/-18V -> Net-(R14-Pad1)
- R14 pad 2: Net-(C28-Pad1) -> +3V3
- R15 pad 1: Net-(C27-Pad2) -> Net-(R15-Pad1)
- R15 pad 2: GND -> +3V3
- R19 pad 1: Net-(C42-Pad2) -> GNDD
- R2 pad 2: GND -> GNDD
- R21 pad 1: Net-(C46-Pad2) -> GNDD
- R6 pad 1: /AK4452DAC/~PDN -> /USB/~RST
- U1 pad 1: /USB/~CS -> +3V3
- U1 pad 2: Net-(U1-Pad2) -> GNDD
- U1 pad 3: Net-(U1-Pad3) -> /USB/MCLK_INT
- U1 pad 4: GND -> Net-(U1-Pad4)
- U1 pad 6: /USB/CLK -> Net-(U1-Pad6)
- U1 pad 7: Net-(U1-Pad7) -> (no net)
- U1 pad 8: +3V3 -> GNDD
- U1 pad 9: (no net) -> GND
- U10 pad 1: +15V -> -12V
- U10 pad 2: GND -> Net-(C24-Pad2)
- U10 pad 3: GND -> Net-(C24-Pad2)
- U10 pad 5: Net-(U10-Pad5) -> GND
- U10 pad 6: GND -> Net-(C24-Pad2)
- U10 pad 7: GND -> Net-(C24-Pad2)
- U10 pad 8: /Power Supply/+18V -> Net-(U10-Pad8)
- U11 pad 1: -12VA -> GND
- U11 pad 2: /Power Supply/-18V -> +3.3VA
- U11 pad 3: /Power Supply/-18V -> VCC
- U12 pad 1: Net-(C42-Pad2) -> GNDD
- U12 pad 3: +3V3 -> VBUS
- U12 pad 5: +3V3 -> VBUS
- U13 pad 1: Net-(C46-Pad2) -> GNDD
- U13 pad 3: +3V3 -> VBUS
- U14 pad 10: GND -> GNDD
- U14 pad 11: +3V3 -> +3.3VA
- U14 pad 12: +3V3 -> +3.3VA
- U14 pad 13: +3V3 -> +3.3VA
- U14 pad 15: Net-(R23-Pad2) -> Net-(R22-Pad2)
- U14 pad 28: +3V3 -> +3.3VA
- U14 pad 29: +3V3 -> +3.3VA
- U14 pad 30: GND -> GNDD
- U14 pad 8: GND -> GNDD
- U14 pad 9: GND -> GNDD
- U3 pad 1: /AK4452DAC/LRCK -> Net-(U1-Pad4)
- U3 pad 11: /USB/~CS -> Net-(U3-Pad11)
- U3 pad 12: /USB/CLK -> Net-(U3-Pad12)
- U3 pad 15: Net-(U1-Pad5) -> Net-(R1-Pad1)
- U3 pad 17: Net-(U1-Pad2) -> Net-(R13-Pad1)
- U3 pad 18: Net-(U1-Pad3) -> Net-(R14-Pad1)
- U3 pad 19: Net-(U1-Pad7) -> Net-(R15-Pad1)
- U3 pad 2: /AK4452DAC/DIN -> Net-(U1-Pad5)
- U3 pad 23: Net-(J1-Pad1) -> VBUS
- U3 pad 4: /USB/BCLK -> Net-(U1-Pad6)
- U3 pad 54: GND -> GNDD
- U3 pad 57: /AK4452DAC/~PDN -> /USB/~RST
- U3 pad 58: Net-(U2-Pad4) -> Net-(U3-Pad58)
- U3 pad 64: /AK4452DAC/MCLK -> /USB/MCLK_INT
- U3 pad 65: GND -> GNDD
- U4 pad 1: /AK4452DAC/~PDN -> /USB/~RST
- U4 pad 3: GND -> GNDD
- U5 pad 1: +3V3 -> /USB/SPDIF
- U5 pad 2: /USB/SPDIF -> /USB/MCLK_INT
- U5 pad 3: /AK4452DAC/MCLK -> GNDD
- U5 pad 4: +3V3 -> Net-(R11-Pad2)
- U5 pad 5: Net-(R11-Pad2) -> +3V3
- U6 pad 1: /USB/CSEL -> Net-(U6-Pad1)
- U6 pad 2: Net-(U2-Pad10) -> Net-(U6-Pad2)
- U6 pad 4: /AK4452DAC/MCLK -> (no net)
- U6 pad 5: Net-(U6-Pad5) -> /USB/MCLK_INT
- U6 pad 6: Net-(U6-Pad6) -> /USB/CSEL
- U6 pad 7: Net-(U6-Pad7) -> GNDD
- U6 pad 8: GND -> +3V3
- U7 pad 1: Net-(D2-Pad2) -> VCC
- U7 pad 3: Net-(C27-Pad2) -> Net-(C22-Pad1)
- U7 pad 4: Net-(R13-Pad1) -> GND
- U7 pad 5: +3V3 -> Net-(C24-Pad2)
- U8 pad 1: Net-(C24-Pad2) -> +12V
- U8 pad 2: Net-(C24-Pad2) -> GND
- U8 pad 3: Net-(C24-Pad1) -> GND
- U8 pad 4: Net-(C22-Pad1) -> Net-(U8-Pad4)
- U8 pad 5: GND -> Net-(U8-Pad5)
- U8 pad 6: Net-(U8-Pad6) -> GND
- U8 pad 7: Net-(U8-Pad7) -> GND
- U8 pad 8: Net-(U8-Pad8) -> Net-(C22-Pad1)
- U9 pad 8: +3V3 -> VCC
- Y1 pad 1: Net-(C5-Pad1) -> Net-(Y1-Pad1)
- Y1 pad 2: Net-(C7-Pad1) -> GNDD
- Y2 pad 1: Net-(C16-Pad1) -> Net-(Y2-Pad1)
- Y2 pad 2: Net-(C18-Pad1) -> GNDD
- Y3 pad 2: Net-(C19-Pad1) -> GNDD
Other:
- board outline added: 106.7 x 109.9 mm
- rule pad_to_mask_clearance: 0.2 -> 0
- board text added: "BACK"
- board text added: "FRONT"

Commit message: Fixed gitignore issue which leaves out the component cache
Parts:
- moved R35 185.6 mm to (117.4, 126.7)
- moved R37 185.6 mm to (122.5, 126.7)
- moved R38 185.6 mm to (117.4, 132.2)
- moved C49 184.9 mm to (179.9, 104.3)
- moved C54 184.9 mm to (170.0, 104.3)
- moved C56 184.9 mm to (174.9, 104.3)
- moved C57 184.9 mm to (168.5, 109.8)
- moved C58 184.9 mm to (155.6, 124.4)
- moved C59 184.9 mm to (150.7, 122.9)
- moved C61 184.9 mm to (173.4, 109.8)
- moved C62 184.9 mm to (168.5, 115.4)
- moved C63 184.9 mm to (132.1, 127.9)
- moved C65 184.9 mm to (132.1, 122.4)
- moved R25 184.9 mm to (178.9, 120.8)
- moved R26 184.9 mm to (184.9, 104.2)
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
Commit message: updated to new kicad format
Changed lines of the file:
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@@
-(kicad_pcb (version 4) (host pcbnew 4.0.6)
+(kicad_pcb (version 20171130) (host pcbnew "(2018-01-27 revision f4273b9e4)-master")
   (general
-    (links 312)
-    (no_connects 312)
-    (area 88.849999 50.749999 195.630001 160.705001)
     (thickness 1.6)
     (drawings 8)
@@
       (layerselection 0x00030_80000001)
       (usegerberextensions false)
+      (usegerberattributes false)
+      (usegerberadvancedattributes false)
+      (creategerberjobfile false)
       (excludeedgelayer true)
       (linewidth 0.100000)
@@
       (hpglpenspeed 20)
       (hpglpendiameter 15)
-      (hpglpenoverlay 2)
       (psnegative false)
       (psa4output false)
@@
     (add_net VCC)
   )
+  (module dacparts:PTR90 (layer F.Cu)
+    (at 102.91 154.94)
+    (fp_text reference RV1 (at 0.5 -4) (layer F.SilkS)
+      (effects (font (size 1 1) (thickness 0.15)))
+    )
+    (fp_text value P10K (at 0 -2.5) (layer F.Fab)
+      (effects (font (size 1 1) (thickness 0.15)))
+    )
+    (fp_line (start 5.08 -8.255) (end 5.08 -7.62) (layer F.SilkS) (width 0.15))
+    (fp_line (start -4.445 -8.255) (end 5.08 -8.255) (layer F.SilkS) (width 0.15))
+    (fp_line (start -4.445 -7.62) (end -4.445 -8.255) (layer F.SilkS) (width 0.15))
+    (fp_line (start -4.445 -7.62) (end -4.445 5.08) (layer F.SilkS) (width 0.15))
+    (fp_line (start 5.08 5.08) (end -4.445 5.08) (layer F.SilkS) (width 0.15))
+    (fp_line (start 5.08 -7.62) (end 5.08 5.08) (layer F.SilkS) (width 0.15))
+    (pad 1 thru_hole circle (at -2.5 0) (size 2 2) (drill 1) (layers *.Cu *.Mask)
+      (net 2 GND))
+    (pad 5 thru_hole circle (at 0 2.5) (size 2 2) (drill 1) (layers *.Cu *.Mask)
+      (net 66 "/Balanced Out/INR"))
+    (pad 6 thru_hole circle (at 2.5 2.5) (size 2 2) (drill 1) (layers *.Cu *.Mask)
+      (net 29 /AK4452DAC/OUTR))
+    (pad 4 thru_hole circle (at -2.5 2.5) (size 2 2) (drill 1) (layers *.Cu *.Mask)
+      (net 2 GND))
+    (pad 2 thru_hole circle (at 0 0) (size 2 2) (drill 1) (layers *.Cu *.Mask)
+      (net 69 "/Balanced Out/INL"))
+    (pad 3 thru_hole circle (at 2.5 0) (size 2 2) (drill 1) (layers *.Cu *.Mask)
+      (net 27 /AK4452DAC/OUTL))
+    (pad 7 thru_hole circle (at -2.5 -6.25) (size 2 2) (drill 1) (layers *.Cu *.Mask))
+    (pad 8 thru_hole circle (at 2.5 -6.25) (size 2 2) (drill 1) (layers *.Cu *.Mask))
+    (model ${KIPRJMOD}/dacparts.3dshapes/ptr90.wrl
+      (at (xyz 0 0 0))
+      (scale (xyz 1 1 1))
+      (rotate (xyz 0 0 0))
+    )
+  )
   (module Capacitors_SMD:C_0805_HandSoldering (layer F.Cu)
     (at 104.14 121.92)
@@
       (net 4 GNDD))
     (model ${KISYS3DMOD}/Connectors.3dshapes/USB_B.wrl
-      (at (xyz 0.18 -0.05 0))
+      (offset (xyz 4.571999931335449 -1.269999980926514 0))
       (scale (xyz 0.39 0.39 0.39))
       (rotate (xyz 0 0 -90))
@@
     (pad "" np_thru_hole oval (at -6 -8.75 180) (size 2 4) (drill oval 2 4) (layers *.Cu *.Mask))
     (model pjras1x1s_series.wrl
-      (at (xyz 0 0 0.25))
+      (offset (xyz 0 0 6.349999904632568))
       (scale (xyz 0.393701 0.393701 0.393701))
       (rotate (xyz 180 0 0))
@@
     (descr "DC Barrel Jack")
     (tags "Power Jack")
-    (fp_text reference J3 (at -8.45 5.75 450) (layer F.SilkS)
+    (fp_text reference J3 (at -8.45 5.75 90) (layer F.SilkS)
       (effects (font (size 1 1) (thickness 0.15)))
     )
@@
       (net 2 GND))
     (model ${KISYS3DMOD}/Connectors.3dshapes/NMJ6HCD2.wrl
-      (at (xyz 0.32 0.17 0))
+      (offset (xyz 8.127999877929687 4.317999935150147 0))
       (scale (xyz 0.39 0.39 0.39))
       (rotate (xyz -90 0 180))
@@
       (net 2 GND))
     (model ${KISYS3DMOD}/Connectors.3dshapes/NMJ6HCD2.wrl
-      (at (xyz 0.32 0.17 0))
+      (offset (xyz 8.127999877929687 4.317999935150147 0))
       (scale (xyz 0.39 0.39 0.39))
       (rotate (xyz -90 0 180))
@@
       (net 52 "Net-(J6-Pad1)"))
     (model ${KISYS3DMOD}/Connectors.3dshapes/NMJ6HCD2.wrl
-      (at (xyz 0.32 0.17 0))
+      (offset (xyz 8.127999877929687 4.317999935150147 0))
       (scale (xyz 0.39 0.39 0.39))
       (rotate (xyz -90 0 180))
@@
     )
   )
-  (module dacparts:PTR90 (layer F.Cu)
-    (at 102.91 154.94)
-    (fp_text reference RV1 (at 0.5 -4) (layer F.SilkS)
-      (effects (font (size 1 1) (thickness 0.15)))
-    )
-    (fp_text value P10K (at 0 -2.5) (layer F.Fab)
-      (effects (font (size 1 1) (thickness 0.15)))
-    )
-    (pad 8 thru_hole circle (at 2.5 -6.25) (size 2 2) (drill 1) (layers *.Cu *.Mask))
-    (pad 7 thru_hole circle (at -2.5 -6.25) (size 2 2) (drill 1) (layers *.Cu *.Mask))
-    (pad 3 thru_hole circle (at 2.5 0) (size 2 2) (drill 1) (layers *.Cu *.Mask)
-      (net 27 /AK4452DAC/OUTL))
-    (pad 2 thru_hole circle (at 0 0) (size 2 2) (drill 1) (layers *.Cu *.Mask)
-      (net 69 "/Balanced Out/INL"))
-    (pad 4 thru_hole circle (at -2.5 2.5) (size 2 2) (drill 1) (layers *.Cu *.Mask)
-      (net 2 GND))
-    (pad 6 thru_hole circle (at 2.5 2.5) (size 2 2) (drill 1) (layers *.Cu *.Mask)
-      (net 29 /AK4452DAC/OUTR))
-    (pad 5 thru_hole circle (at 0 2.5) (size 2 2) (drill 1) (layers *.Cu *.Mask)
-      (net 66 "/Balanced Out/INR"))
-    (pad 1 thru_hole circle (at -2.5 0) (size 2 2) (drill 1) (layers *.Cu *.Mask)
-      (net 2 GND))
-  )
   (module Housings_SOIC:SOIC-16W_7.5x10.3mm_Pitch1.27mm (layer F.Cu)

Commit message: started routing PCB
Parts:
- C1, C10, C11, C12, C14, C15, C16, C20, C21, C25, C26, C27, C3, C31, C33, C34, C39, C4, C40, C49, C5, C51, C53, C55, C56, C57, C58, C59, C6, C60, C61, C62, C63, C64, C65, C66, C7, C8, C9: footprint Capacitors_SMD:C_0805_HandSoldering -> Capacitors_SMD:C_0402
- C13, C2, C22, C24, C41, C42, C45, C46, C50, C54: footprint Capacitors_SMD:C_0805_HandSoldering -> Capacitors_SMD:C_0805
- C43, C44, C47, C48, C52: footprint Capacitors_SMD:C_0805_HandSoldering -> Capacitors_SMD:C_1206
- J4, J5, J6: value JACK_TRS_6PINS -> Audio-Jack-3_3Switches
- R1, R11, R12, R13, R14, R15, R18, R19, R20, R21, R22, R23, R24, R25, R26, R27, R28, R29, R30, R31, R32, R33, R35, R37, R38, R39, R6: footprint Resistors_SMD:R_0805_HandSoldering -> Resistors_SMD:R_0402
- R2, R34, R36, R40, R41, R5: footprint Resistors_SMD:R_0805_HandSoldering -> Resistors_SMD:R_0805
- moved C48 130.3 mm to (24.3, 123.8), turned to 270 degrees
- moved R21 122.2 mm to (41.7, 126.7), turned to 180 degrees
- moved R18 119.2 mm to (47.4, 104.3), turned to 180 degrees
- moved R19 115.5 mm to (54.2, 103.8), turned to 180 degrees
- moved C44 97.4 mm to (37.7, 99.6), turned to 270 degrees
- moved C47 87.7 mm to (26.8, 119.6), turned to 180 degrees
- moved R20 86.6 mm to (34.4, 126.7), turned to 180 degrees
- moved C46 86.6 mm to (28.3, 123.1), turned to 270 degrees
- moved L4 81.6 mm to (33.5, 121.8), turned to 90 degrees
- moved U12 74.6 mm to (52.5, 101.1)
- moved C41 74.2 mm to (52.8, 97.9)
- moved U13 72.8 mm to (40.0, 123.9)
- moved L3 72.6 mm to (45.7, 98.8), turned to 90 degrees
- moved C45 72.3 mm to (40.0, 120.0), turned to 180 degrees
- moved C42 70.2 mm to (40.9, 99.1), turned to 270 degrees
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Connections:
- net Net-(J1-Pad2) renamed /USB/D-
- net Net-(J1-Pad3) renamed /USB/D+
- C1 pad 1: VCC -> +3V3
- C10 pad 2: GNDD -> GND
- C11 pad 2: GNDD -> GND
- C12 pad 2: GNDD -> GND
- C13 pad 2: GNDD -> GND
- C14 pad 2: GNDD -> GND
- C15 pad 2: GNDD -> GND
- C16 pad 2: GNDD -> GND
- C2 pad 2: GNDD -> GND
- C21 pad 1: GNDD -> GND
- C23 pad 1: VCC -> +3V3
- C25 pad 1: VCC -> +3V3
- C26 pad 1: VCC -> +3V3
- C3 pad 2: GNDD -> GND
- C4 pad 2: GNDD -> GND
- C42 pad 2: GNDD -> GND
- C43 pad 2: GNDD -> GND
- C44 pad 2: GNDD -> GND
- C46 pad 2: GNDD -> GND
- C47 pad 2: GNDD -> GND
- C48 pad 2: GNDD -> GND
- C5 pad 2: GNDD -> GND
- C51 pad 2: GNDD -> GND
- C52 pad 2: GNDD -> GND
- C53 pad 2: GNDD -> GND
- C54 pad 1: GNDD -> GND
- C6 pad 2: GNDD -> GND
- C63 pad 1: +15V -> +12V
- C64 pad 2: -12VA -> -12V
- C65 pad 1: +15V -> +12V
- C66 pad 2: -12VA -> -12V
- C7 pad 2: GNDD -> GND
- C8 pad 2: GNDD -> GND
- C9 pad 2: GNDD -> GND
- D1 pad 1: VCC -> +3V3
- J1 pad 4: GNDD -> GND
- J1 pad 5: GNDD -> GND
- J2 pad 2: GNDD -> GND
- J4 pad 1: GND -> (no net)
- J4 pad 2: Net-(J4-Pad2) -> (no net)
- J4 pad 3: Net-(J4-Pad3) -> GND
- J4 pad 4: GND -> Net-(J4-Pad4)
- J4 pad 6: Net-(J4-Pad6) -> GND
- J5 pad 1: GND -> (no net)
- J5 pad 2: Net-(J5-Pad2) -> (no net)
- J5 pad 3: Net-(J5-Pad3) -> GND
- J5 pad 4: GND -> Net-(J5-Pad4)
- J5 pad 6: Net-(J5-Pad6) -> GND
- J6 pad 4: Net-(J6-Pad4) -> (no net)
- J6 pad 6: Net-(J6-Pad6) -> (no net)
- R12 pad 1: GNDD -> GND
- R19 pad 1: GNDD -> GND
- R2 pad 2: GNDD -> GND
- R21 pad 1: GNDD -> GND
- R22 pad 2: Net-(R22-Pad2) -> (no net)
- U1 pad 2: GNDD -> GND
- U1 pad 8: GNDD -> GND
- U10 pad 4: Net-(U10-Pad4) -> (no net)
- U10 pad 8: Net-(U10-Pad8) -> (no net)
- U11 pad 3: VCC -> +3V3
- U12 pad 1: GNDD -> GND
- U13 pad 1: GNDD -> GND
- U14 pad 10: GNDD -> GND
- U14 pad 15: Net-(R22-Pad2) -> Net-(R23-Pad2)
- U14 pad 30: GNDD -> GND
- U14 pad 32: /AK4452DAC/~PDN -> (no net)
- U14 pad 6: Net-(U14-Pad6) -> (no net)
- U14 pad 7: /AK4452DAC/MUTE -> (no net)
- U14 pad 8: GNDD -> GND
- U14 pad 9: GNDD -> GND
- U15 pad 1: Net-(U15-Pad1) -> (no net)
- U15 pad 4: -12VA -> -12V
- U15 pad 7: +15V -> +12V
- U16 pad 1: Net-(U16-Pad1) -> (no net)
- U16 pad 4: -12VA -> -12V
- U16 pad 7: +15V -> +12V
- U17 pad 1: Net-(J5-Pad3) -> Net-(J5-Pad4)
- U17 pad 2: Net-(J5-Pad3) -> Net-(J5-Pad4)
- U17 pad 5: -12VA -> -12V
- U17 pad 6: +15V -> +12V
- U17 pad 7: Net-(J5-Pad2) -> Net-(J5-Pad5)
- U17 pad 8: Net-(J5-Pad2) -> Net-(J5-Pad5)
- U18 pad 1: Net-(J4-Pad3) -> Net-(J4-Pad4)
- U18 pad 2: Net-(J4-Pad3) -> Net-(J4-Pad4)
- U18 pad 5: -12VA -> -12V
- U18 pad 6: +15V -> +12V
- U18 pad 7: Net-(J4-Pad2) -> Net-(J4-Pad5)
- U18 pad 8: Net-(J4-Pad2) -> Net-(J4-Pad5)
- U19 pad 1: -12VA -> -12V
- U19 pad 18: +15V -> +12V
- U19 pad 20: -12VA -> -12V
- U19 pad 3: +15V -> +12V
- U3 pad 11: Net-(U3-Pad11) -> (no net)
- U3 pad 12: Net-(U3-Pad12) -> (no net)
- U3 pad 14: Net-(U3-Pad14) -> (no net)
- U3 pad 16: Net-(U3-Pad16) -> (no net)
- U3 pad 21: Net-(U3-Pad21) -> (no net)
- U3 pad 28: Net-(U3-Pad28) -> (no net)
- U3 pad 29: Net-(U3-Pad29) -> (no net)
- U3 pad 30: Net-(U3-Pad30) -> (no net)
- U3 pad 32: Net-(U3-Pad32) -> (no net)
- U3 pad 33: Net-(U3-Pad33) -> (no net)
- U3 pad 35: Net-(U3-Pad35) -> (no net)
- U3 pad 36: Net-(U3-Pad36) -> (no net)
- U3 pad 37: Net-(U3-Pad37) -> (no net)
- U3 pad 43: Net-(U3-Pad43) -> (no net)
- U3 pad 45: Net-(U3-Pad45) -> (no net)
- U3 pad 46: Net-(U3-Pad46) -> (no net)
- U3 pad 47: Net-(U3-Pad47) -> (no net)
- U3 pad 48: Net-(U3-Pad48) -> (no net)
- U3 pad 49: Net-(U3-Pad49) -> (no net)
- U3 pad 5: Net-(U3-Pad5) -> (no net)
- U3 pad 50: Net-(U3-Pad50) -> (no net)
- U3 pad 51: Net-(U3-Pad51) -> (no net)
- U3 pad 54: GNDD -> GND
- U3 pad 6: Net-(U3-Pad6) -> (no net)
- U3 pad 60: Net-(U3-Pad60) -> (no net)
- U3 pad 61: Net-(U3-Pad61) -> (no net)
- U3 pad 62: Net-(U3-Pad62) -> (no net)
- U3 pad 63: Net-(U3-Pad63) -> (no net)
- U3 pad 65: GNDD -> GND
- U3 pad 7: Net-(U3-Pad7) -> (no net)
- U3 pad 8: Net-(U3-Pad8) -> (no net)
- U4 pad 3: GNDD -> GND
- U5 pad 3: GNDD -> GND
- U6 pad 3: Net-(U6-Pad3) -> (no net)
- U6 pad 7: GNDD -> GND
- U7 pad 1: VCC -> +3V3
- U8 pad 4: Net-(U8-Pad4) -> (no net)
- U8 pad 5: Net-(U8-Pad5) -> (no net)
- U9 pad 4: Net-(U9-Pad4) -> (no net)
- U9 pad 5: Net-(U9-Pad5) -> (no net)
- U9 pad 8: VCC -> +3V3
- Y1 pad 1: Net-(Y1-Pad1) -> (no net)
- Y1 pad 2: GNDD -> GND
- Y2 pad 1: Net-(Y2-Pad1) -> (no net)
- Y2 pad 2: GNDD -> GND
- Y3 pad 1: Net-(Y3-Pad1) -> (no net)
- Y3 pad 2: GNDD -> GND
Routing:
- net Net-(C20-Pad1): track 0.00 -> 6.55 mm
- net Net-(R11-Pad2): track 0.00 -> 4.84 mm
- net Net-(C20-Pad2): track 0.00 -> 1.44 mm
Other:
- net class Power added: clearance 0.3, trace_width 0.375, via_dia 0.6, via_drill 0.4
- net class PowerLV added: clearance 0.4, trace_width 0.5, via_dia 0.8, via_drill 0.6
