File: USB-DAC.sch (KiCad schematic (older format))
At the start: 1 part

Commit message: Updated schematics and part number fields
Parts:
- RV1: value POT_Dual -> P10K; mpn (none) -> PTR902-2020K-A103
Changed lines of the file:
@@
 P 4400 2150
 F 0 "RV1" H 4400 2300 50  0000 C CNN
-F 1 "POT_Dual" H 4400 2225 50  0000 C CNN
+F 1 "P10K" H 4400 2225 50  0000 C CNN
 F 2 "" H 4650 2075 50  0001 C CNN
 F 3 "" H 4650 2075 50  0001 C CNN
+F 4 "PTR902-2020K-A103" H 4400 2150 60  0001 C CNN "mpn"
 	1    4400 2150
 	0    1    1    0
@@
 	4200 1750 4300 1750
 $Comp
-L GND #PWR01
+L GND #PWR1
 U 1 1 5A0F0FC7
 P 4300 1500
-F 0 "#PWR01" H 4300 1250 50  0001 C CNN
+F 0 "#PWR1" H 4300 1250 50  0001 C CNN
 F 1 "GND" H 4300 1350 50  0000 C CNN
 F 2 "" H 4300 1500 50  0001 C CNN

Commit message: Began PCB layout
Parts:
- RV1: footprint (none) -> dacparts:PTR90
Changed lines of the file:
@@
 $EndDescr
-$Sheet
-S 1950 1750 750  800
-U 59E908E3
-F0 "USB" 60
-F1 "file59E908E2.sch" 60
-F2 "MCLK" O R 2700 1850 60
-F3 "LRCK" O R 2700 2050 60
-F4 "DOUT" O R 2700 2150 60
-F5 "BCLK" O R 2700 1950 60
-F6 "~RST" I R 2700 2250 60
-$EndSheet
 $Sheet
 S 2100 3650 1000 850
@@
 Wire Wire Line
 	3100 2150 2700 2150
-Wire Wire Line
-	2700 2250 2900 2250
-Wire Wire Line
-	2900 2250 2900 2350
-Wire Wire Line
-	2900 2350 3100 2350
 $Sheet
 S 5100 2600 1450 800
@@
 F 0 "RV1" H 4400 2300 50  0000 C CNN
 F 1 "P10K" H 4400 2225 50  0000 C CNN
-F 2 "" H 4650 2075 50  0001 C CNN
+F 2 "dacparts:PTR90" H 4650 2075 50  0001 C CNN
 F 3 "" H 4650 2075 50  0001 C CNN
 F 4 "PTR902-2020K-A103" H 4400 2150 60  0001 C CNN "mpn"
@@
 	4200 1750 4300 1750
 $Comp
-L GND #PWR1
+L GND #PWR01
 U 1 1 5A0F0FC7
 P 4300 1500
-F 0 "#PWR1" H 4300 1250 50  0001 C CNN
+F 0 "#PWR01" H 4300 1250 50  0001 C CNN
 F 1 "GND" H 4300 1350 50  0000 C CNN
 F 2 "" H 4300 1500 50  0001 C CNN
@@
 	4500 2400 5000 2400
 Connection ~ 5000 2400
+$Sheet
+S 1950 1750 750  800
+U 59E908E3
+F0 "USB" 60
+F1 "file59E908E2.sch" 60
+F2 "MCLK" O R 2700 1850 60
+F3 "LRCK" O R 2700 2050 60
+F4 "DOUT" O R 2700 2150 60
+F5 "BCLK" O R 2700 1950 60
+F6 "~RST" I R 2700 2250 60
+$EndSheet
 $EndSCHEMATC

Commit message: updated to new kicad format
Parts:
- RV1: symbol POT_Dual -> Device:POT_Dual
Changed lines of the file:
@@
-EESchema Schematic File Version 2
-LIBS:power
-LIBS:device
-LIBS:transistors
-LIBS:conn
-LIBS:linear
-LIBS:regul
-LIBS:74xx
-LIBS:cmos4000
-LIBS:adc-dac
-LIBS:memory
-LIBS:xilinx
-LIBS:microcontrollers
-LIBS:dsp
-LIBS:microchip
-LIBS:analog_switches
-LIBS:motorola
-LIBS:texas
-LIBS:intel
-LIBS:audio
-LIBS:interface
-LIBS:digital-audio
-LIBS:philips
-LIBS:display
-LIBS:cypress
-LIBS:siliconi
-LIBS:opto
-LIBS:atmel
-LIBS:contrib
-LIBS:valves
-LIBS:dacparts
-LIBS:USB-DAC-cache
-EELAYER 25 0
+EESchema Schematic File Version 4
+EELAYER 26 0
 EELAYER END
 $Descr A4 11693 8268
@@
 $EndSheet
 $Comp
-L POT_Dual RV1
+L Device:POT_Dual RV1
 U 1 1 5A0F0848
 P 4400 2150
@@
 	4200 2250 4300 2250
 Wire Wire Line
-	4200 1500 4200 2250
+	4200 1500 4200 1750
 Wire Wire Line
 	4200 1750 4300 1750
 $Comp
-L GND #PWR01
+L power:GND #PWR01
 U 1 1 5A0F0FC7
 P 4300 1500
@@
 	4200 2550 4300 2550
 Wire Wire Line
-	4500 1900 5100 1900
+	4500 1900 4900 1900
 Wire Wire Line
 	4900 1900 4900 2850
@@
 	5100 2200 5000 2200
 Wire Wire Line
-	5000 2200 5000 3150
+	5000 2200 5000 2400
 Wire Wire Line
 	5000 3150 5100 3150
@@
 F6 "~RST" I R 2700 2250 60
 $EndSheet
+Wire Wire Line
+	4200 1750 4200 2250
+Wire Wire Line
+	4900 1900 5100 1900
+Wire Wire Line
+	5000 2400 5000 3150
 $EndSCHEMATC

Commit message: started routing PCB
Connections:
- no-connect marks 0 -> 1
Changed lines of the file:
@@
 EESchema Schematic File Version 4
+LIBS:USB-DAC-cache
 EELAYER 26 0
 EELAYER END
@@
 Wire Wire Line
 	5000 2400 5000 3150
+NoConn ~ 5300 8050
 $EndSCHEMATC
