File: file59E908E2.sch (KiCad schematic (older format))
At the start: 44 parts, among them J1 USB_B, J2 SPDIF OUT, U1 S25FL116K0XNFA013, U2 74LV14, U3 XHRA-2HPA, U4 NCP303LSN09T1G, U5 74LS74, U6 74LS157, Y1 24, Y2 24.576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

Commit message: Updated schematics and part number fields
Parts:
- J2: mpn (none) -> RCJ-014
- R1, R2, R3: footprint (none) -> Resistors_SMD:R_0805_HandSoldering
- R4: footprint (none) -> Resistors_SMD:R_0805_HandSoldering; MPN (none) -> RC0805FR-07220RL
- R5: footprint (none) -> Resistors_SMD:R_0805_HandSoldering; MPN (none) -> RC0805FR-074R7L
- U1: footprint (none) -> Housings_SON:WSON-8_1EP_2x2mm_Pitch0.5mm
- U2: footprint (none) -> Housings_SOIC:SOIC-14_3.9x8.7mm_Pitch1.27mm; mpn (none) -> SN74LV14ADR
- U2: footprint (none) -> Housings_SOIC:SOIC-14_3.9x8.7mm_Pitch1.27mm
- U3: footprint Housings_QFP:TQFP-64_10x10mm_Pitch0.5mm -> Housings_QFP:TQFP-64-1EP_10x10mm_Pitch0.5mm
- U4: footprint (none) -> TO_SOT_Packages_SMD:SOT-23-5_HandSoldering
- U5: value 74LS74 -> 74LV74; footprint (none) -> Housings_SOIC:SOIC-14_3.9x8.7mm_Pitch1.27mm; mpn (none) -> SN74LV74ADR
- U6: value 74LS157 -> 74LV157; footprint (none) -> Housings_SOIC:SOIC-16_3.9x9.9mm_Pitch1.27mm; mpn (none) -> SN74LV174ADR

Commit message: Began PCB layout
Parts:
- removed C1: 100n, Capacitors_SMD:C_0805_HandSoldering, symbol C_Small
- removed C17, C18, C19: 18p, Capacitors_SMD:C_0805_HandSoldering, symbol C_Small
- removed R10, R4, R9: 220, Resistors_SMD:R_0805_HandSoldering, symbol R
- removed R3, R7, R8: 1M, Resistors_SMD:R_0805_HandSoldering, symbol R
- removed U1: S25FL116K0XNFA013, Housings_SON:WSON-8_1EP_2x2mm_Pitch0.5mm, symbol S25FL116K0XNFA013
- removed U2: 74LV14, Housings_SOIC:SOIC-14_3.9x8.7mm_Pitch1.27mm, symbol 74LV14
- removed U5: 74LV74, Housings_SOIC:SOIC-14_3.9x8.7mm_Pitch1.27mm, symbol 74LS74
- removed U6: 74LV157, Housings_SOIC:SOIC-16_3.9x9.9mm_Pitch1.27mm, symbol 74LS157
- removed Y1: 24, Crystals:Crystal_SMD_HC49-SD_HandSoldering, symbol Crystal
- removed Y2: 24.576, Crystals:Crystal_SMD_HC49-SD_HandSoldering, symbol Crystal
- removed Y3: 22.5792, Crystals:Crystal_SMD_HC49-SD_HandSoldering, symbol Crystal
- added R13, R14, R15: 0, Resistors_SMD:R_0805_HandSoldering, symbol R
- added U1: ISO7340FC, Housings_SOIC:SOIC-16W_7.5x10.3mm_Pitch1.27mm, symbol ISO7340FC
- added U5: 74LVC1G79, TO_SOT_Packages_SMD:SOT-353_SC-70-5_Handsoldering, symbol 74LVC1G79
- added U6: TC7WH157, Housings_SSOP:SSOP-8_2.95x2.8mm_Pitch0.65mm, symbol TC7WH157
- added Y1: 24, Crystals:Crystal_SMD_3225-4pin_3.2x2.5mm, symbol Crystal_GND24
- added Y2: 24.576, Crystals:Crystal_SMD_3225-4pin_3.2x2.5mm, symbol Crystal_GND24
- added Y3: 22.5792, Crystals:Crystal_SMD_2016-4pin_2.0x1.6mm, symbol Crystal_GND24
- C13: mpn CL21B106KPQNNNE -> (none)
- C16: value 18p -> 100n; mpn CL21C180JBANNNC -> (none)
- C5, C7: value 18p -> 100n
- J2: footprint (none) -> dacparts:pjras1x1s_series; mpn RCJ-014 -> PJRAS1X1S04X
- R1: value 10K -> 0
- R2: mpn (none) -> RC0805FR-0743R2L
- R6: mpn (none) -> RC0805FR-071KL
Connections:
- net labels added: +3.3VA, GND, MCLK_INT, VBUS
- net labels removed: CLK, ~CS
- wire segments 169 -> 163
- no-connect marks 0 -> 1
Other:
- note added: "* pin 1 may need gnd connection\n"
- note added: "*Actually an oscillator"
- moved on the sheet: C20, C21, J2, R11, R12

Commit message: updated to new kicad format
Parts:
- C10, C11, C12, C13, C14, C15, C16, C2, C20, C21, C3, C4, C5, C6, C7, C8, C9: symbol C_Small -> Device:C_Small
- J1: symbol USB_B -> Connector_Specialized:USB_B
- J2: symbol CONN_COAXIAL -> Connector_Specialized:Conn_Coaxial
- R1, R11, R12, R13, R14, R15, R2, R5, R6: symbol R -> Device:R
- U1: symbol ISO7340FC -> Isolator:ISO7340FC
- U3: symbol XHRA-2HPA -> dacparts:XHRA-2HPA
- U4: symbol NCP303LSN09T1G -> dacparts:NCP303LSN09T1G
- U5: symbol 74LVC1G79 -> Logic_74xgxx:74LVC1G79
- U6: symbol TC7WH157 -> dacparts:TC7WH157
- Y1, Y2, Y3: symbol Crystal_GND24 -> Device:Crystal_GND24
Connections:
- wire segments 163 -> 207
Other:
- moved on the sheet: U5

Commit message: started routing PCB
Parts:
- C10, C11, C12, C14, C15, C16, C20, C21, C3, C4, C5, C6, C7, C8, C9: footprint Capacitors_SMD:C_0805_HandSoldering -> Capacitors_SMD:C_0402
- C13, C2: footprint Capacitors_SMD:C_0805_HandSoldering -> Capacitors_SMD:C_0805
- R1, R11, R12, R13, R14, R15, R6: footprint Resistors_SMD:R_0805_HandSoldering -> Resistors_SMD:R_0402
- R2, R5: footprint Resistors_SMD:R_0805_HandSoldering -> Resistors_SMD:R_0805
Connections:
- net labels added: D+, D-
- wire segments 207 -> 208
- no-connect marks 1 -> 24
Changed lines of the file:
@@
 EESchema Schematic File Version 4
+LIBS:USB-DAC-cache
 EELAYER 26 0
 EELAYER END
@@
 F 0 "C9" H 8360 3820 50  0000 L CNN
 F 1 "100n" H 8360 3670 50  0000 L CNN
-F 2 "Capacitors_SMD:C_0805_HandSoldering" H 8350 3750 50  0001 C CNN
+F 2 "Capacitors_SMD:C_0402" H 8350 3750 50  0001 C CNN
 F 3 "" H 8350 3750 50  0001 C CNN
 	1    8350 3750
@@
 L power:+1V0 #PWR058
 U 1 1 59E91219
-P 6750 5450
-F 0 "#PWR058" H 6750 5300 50  0001 C CNN
-F 1 "+1V0" H 6900 5500 50  0000 C CNN
-F 2 "" H 6750 5450 50  0001 C CNN
-F 3 "" H 6750 5450 50  0001 C CNN
-	1    6750 5450
+P 6750 5400
+F 0 "#PWR058" H 6750 5250 50  0001 C CNN
+F 1 "+1V0" H 6900 5450 50  0000 C CNN
+F 2 "" H 6750 5400 50  0001 C CNN
+F 3 "" H 6750 5400 50  0001 C CNN
+	1    6750 5400
 	1    0    0    -1
 $EndComp
@@
 F 0 "R2" V 6700 5000 50  0000 C CNN
 F 1 "43.2" V 6750 5150 50  0000 C CNN
-F 2 "Resistors_SMD:R_0805_HandSoldering" V 6680 5150 50  0001 C CNN
+F 2 "Resistors_SMD:R_0805" V 6680 5150 50  0001 C CNN
 F 3 "" H 6750 5150 50  0001 C CNN
 F 4 "RC0805FR-0743R2L" V 6750 5150 60  0001 C CNN "mpn"
@@
 F 0 "R5" V 9430 4100 50  0000 C CNN
 F 1 "4.7" V 9350 4100 50  0000 C CNN
-F 2 "Resistors_SMD:R_0805_HandSoldering" V 9280 4100 50  0001 C CNN
+F 2 "Resistors_SMD:R_0805" V 9280 4100 50  0001 C CNN
 F 3 "" H 9350 4100 50  0001 C CNN
 F 4 "RC0805FR-074R7L" V 9350 4100 60  0001 C CNN "MPN"
@@
 F 0 "C14" H 9610 4320 50  0000 L CNN
 F 1 "100n" H 9610 4170 50  0000 L CNN
-F 2 "Capacitors_SMD:C_0805_HandSoldering" H 9600 4250 50  0001 C CNN
+F 2 "Capacitors_SMD:C_0402" H 9600 4250 50  0001 C CNN
 F 3 "" H 9600 4250 50  0001 C CNN
 	1    9600 4250
@@
 F 0 "C10" H 8610 3820 50  0000 L CNN
 F 1 "100n" H 8610 3670 50  0000 L CNN
-F 2 "Capacitors_SMD:C_0805_HandSoldering" H 8600 3750 50  0001 C CNN
+F 2 "Capacitors_SMD:C_0402" H 8600 3750 50  0001 C CNN
 F 3 "" H 8600 3750 50  0001 C CNN
 	1    8600 3750
@@
 F 0 "C11" H 8860 3820 50  0000 L CNN
 F 1 "100n" H 8860 3670 50  0000 L CNN
-F 2 "Capacitors_SMD:C_0805_HandSoldering" H 8850 3750 50  0001 C CNN
+F 2 "Capacitors_SMD:C_0402" H 8850 3750 50  0001 C CNN
 F 3 "" H 8850 3750 50  0001 C CNN
 	1    8850 3750
@@
 F 0 "C12" H 9110 3820 50  0000 L CNN
 F 1 "100n" H 9110 3670 50  0000 L CNN
-F 2 "Capacitors_SMD:C_0805_HandSoldering" H 9100 3750 50  0001 C CNN
+F 2 "Capacitors_SMD:C_0402" H 9100 3750 50  0001 C CNN
 F 3 "" H 9100 3750 50  0001 C CNN
 	1    9100 3750
@@
 F 0 "C3" H 7360 3820 50  0000 L CNN
 F 1 "100n" H 7360 3670 50  0000 L CNN
-F 2 "Capacitors_SMD:C_0805_HandSoldering" H 7350 3750 50  0001 C CNN
+F 2 "Capacitors_SMD:C_0402" H 7350 3750 50  0001 C CNN
 F 3 "" H 7350 3750 50  0001 C CNN
 F 4 "CL21B104MBCNNNC" H 7350 3750 60  0001 C CNN "mpn"
@@
 F 0 "C4" H 7610 3820 50  0000 L CNN
 F 1 "100n" H 7610 3670 50  0000 L CNN
-F 2 "Capacitors_SMD:C_0805_HandSoldering" H 7600 3750 50  0001 C CNN
+F 2 "Capacitors_SMD:C_0402" H 7600 3750 50  0001 C CNN
 F 3 "" H 7600 3750 50  0001 C CNN
 	1    7600 3750
@@
 F 0 "C6" H 7860 3820 50  0000 L CNN
 F 1 "100n" H 7860 3670 50  0000 L CNN
-F 2 "Capacitors_SMD:C_0805_HandSoldering" H 7850 3750 50  0001 C CNN
+F 2 "Capacitors_SMD:C_0402" H 7850 3750 50  0001 C CNN
 F 3 "" H 7850 3750 50  0001 C CNN
 	1    7850 3750
@@
 F 0 "C8" H 8110 3820 50  0000 L CNN
 F 1 "100n" H 8110 3670 50  0000 L CNN
-F 2 "Capacitors_SMD:C_0805_HandSoldering" H 8100 3750 50  0001 C CNN
+F 2 "Capacitors_SMD:C_0402" H 8100 3750 50  0001 C CNN
 F 3 "" H 8100 3750 50  0001 C CNN
 	1    8100 3750
@@
 F 0 "C13" H 9360 3820 50  0000 L CNN
 F 1 "10u" H 9360 3670 50  0000 L CNN
-F 2 "Capacitors_SMD:C_0805_HandSoldering" H 9350 3750 50  0001 C CNN
+F 2 "Capacitors_SMD:C_0805" H 9350 3750 50  0001 C CNN
 F 3 "" H 9350 3750 50  0001 C CNN
 	1    9350 3750
@@
 F 0 "C2" H 7160 3820 50  0000 L CNN
 F 1 "10u" H 7160 3670 50  0000 L CNN
-F 2 "Capacitors_SMD:C_0805_HandSoldering" H 7150 3750 50  0001 C CNN
+F 2 "Capacitors_SMD:C_0805" H 7150 3750 50  0001 C CNN
 F 3 "" H 7150 3750 50  0001 C CNN
 F 4 "CL21A106KAFN3NE" H 7150 3750 60  0001 C CNN "mpn"
@@
 Wire Wire Line
 	7050 5350 6050 5350
-Wire Wire Line
-	5750 5700 5750 5650
 Wire Wire Line
 	5650 5650 5650 5700
@@
 F 0 "R11" V 12080 2950 50  0000 C CNN
 F 1 "220" V 12000 2950 50  0000 C CNN
-F 2 "Resistors_SMD:R_0805_HandSoldering" V 11930 2950 50  0001 C CNN
+F 2 "Resistors_SMD:R_0402" V 11930 2950 50  0001 C CNN
 F 3 "" H 12000 2950 50  0001 C CNN
 	1    12000 2950
@@
 F 0 "C20" H 12310 3020 50  0000 L CNN
 F 1 "100n" H 12310 2870 50  0000 L CNN
-F 2 "Capacitors_SMD:C_0805_HandSoldering" H 12300 2950 50  0001 C CNN
+F 2 "Capacitors_SMD:C_0402" H 12300 2950 50  0001 C CNN
 F 3 "" H 12300 2950 50  0001 C CNN
 	1    12300 2950
@@
 F 0 "R12" V 12580 3150 50  0000 C CNN
 F 1 "220" V 12500 3150 50  0000 C CNN
-F 2 "Resistors_SMD:R_0805_HandSoldering" V 12430 3150 50  0001 C CNN
+F 2 "Resistors_SMD:R_0402" V 12430 3150 50  0001 C CNN
 F 3 "" H 12500 3150 50  0001 C CNN
 	1    12500 3150
@@
 F 0 "C21" H 12660 3220 50  0000 L CNN
 F 1 "100p" H 12660 3070 50  0000 L CNN
-F 2 "Capacitors_SMD:C_0805_HandSoldering" H 12650 3150 50  0001 C CNN
+F 2 "Capacitors_SMD:C_0402" H 12650 3150 50  0001 C CNN
 F 3 "" H 12650 3150 50  0001 C CNN
 F 4 "CL21C101JBANNNC" H 12650 3150 60  0001 C CNN "mpn"
@@
 F 0 "R6" V 11080 6700 50  0000 C CNN
 F 1 "1K" V 11000 6700 50  0000 C CNN
-F 2 "Resistors_SMD:R_0805_HandSoldering" V 10930 6700 50  0001 C CNN
+F 2 "Resistors_SMD:R_0402" V 10930 6700 50  0001 C CNN
 F 3 "" H 11000 6700 50  0001 C CNN
 F 4 "RC0805FR-071KL" V 11000 6700 60  0001 C CNN "mpn"
@@
 F 0 "C15" H 9710 7270 50  0000 L CNN
 F 1 "100n" H 9710 7120 50  0000 L CNN
-F 2 "Capacitors_SMD:C_0805_HandSoldering" H 9700 7200 50  0001 C CNN
+F 2 "Capacitors_SMD:C_0402" H 9700 7200 50  0001 C CNN
 F 3 "" H 9700 7200 50  0001 C CNN
 	1    9700 7200
@@
 F 0 "R1" V 6150 6350 50  0000 C CNN
 F 1 "0" V 6200 6200 50  0000 C CNN
-F 2 "Resistors_SMD:R_0805_HandSoldering" V 6130 6200 50  0001 C CNN
+F 2 "Resistors_SMD:R_0402" V 6130 6200 50  0001 C CNN
 F 3 "" H 6200 6200 50  0001 C CNN
 	1    6200 6200
@@
 F 0 "R13" V 6150 6450 50  0000 C CNN
 F 1 "0" V 6200 6300 50  0000 C CNN
-F 2 "Resistors_SMD:R_0805_HandSoldering" V 6130 6300 50  0001 C CNN
+F 2 "Resistors_SMD:R_0402" V 6130 6300 50  0001 C CNN
 F 3 "" H 6200 6300 50  0001 C CNN
 	1    6200 6300
@@
 F 0 "R14" V 6150 6550 50  0000 C CNN
 F 1 "0" V 6200 6400 50  0000 C CNN
-F 2 "Resistors_SMD:R_0805_HandSoldering" V 6130 6400 50  0001 C CNN
+F 2 "Resistors_SMD:R_0402" V 6130 6400 50  0001 C CNN
 F 3 "" H 6200 6400 50  0001 C CNN
 	1    6200 6400
@@
 F 0 "R15" V 6150 6650 50  0000 C CNN
 F 1 "0" V 6200 6500 50  0000 C CNN
-F 2 "Resistors_SMD:R_0805_HandSoldering" V 6130 6500 50  0001 C CNN
+F 2 "Resistors_SMD:R_0402" V 6130 6500 50  0001 C CNN
 F 3 "" H 6200 6500 50  0001 C CNN
 	1    6200 6500
@@
 F 0 "C7" H 12260 6920 50  0000 L CNN
 F 1 "100n" H 12260 6770 50  0000 L CNN
-F 2 "Capacitors_SMD:C_0805_HandSoldering" H 12250 6850 50  0001 C CNN
+F 2 "Capacitors_SMD:C_0402" H 12250 6850 50  0001 C CNN
 F 3 "" H 12250 6850 50  0001 C CNN
 	1    12250 6850
@@
 F 0 "C16" H 12310 7970 50  0000 L CNN
 F 1 "100n" H 12310 7820 50  0000 L CNN
-F 2 "Capacitors_SMD:C_0805_HandSoldering" H 12300 7900 50  0001 C CNN
+F 2 "Capacitors_SMD:C_0402" H 12300 7900 50  0001 C CNN
 F 3 "" H 12300 7900 50  0001 C CNN
 	1    12300 7900
@@
 F 0 "C5" H 8410 7320 50  0000 L CNN
 F 1 "100n" H 8410 7170 50  0000 L CNN
-F 2 "Capacitors_SMD:C_0805_HandSoldering" H 8400 7250 50  0001 C CNN
+F 2 "Capacitors_SMD:C_0402" H 8400 7250 50  0001 C CNN
 F 3 "" H 8400 7250 50  0001 C CNN
 	1    8400 7250
@@
 Wire Wire Line
 	11550 4600 11550 4900
+NoConn ~ 7300 6650
+NoConn ~ 7400 6650
+NoConn ~ 7500 6650
+NoConn ~ 7700 6650
+NoConn ~ 7800 6650
+NoConn ~ 7900 6650
+NoConn ~ 8000 6650
+NoConn ~ 8300 6650
+NoConn ~ 8400 6650
+NoConn ~ 8500 6650
+NoConn ~ 8600 6650
+NoConn ~ 8700 6650
+NoConn ~ 8800 6650
+NoConn ~ 8900 6650
+NoConn ~ 9000 6650
+NoConn ~ 7050 4750
+NoConn ~ 7050 4850
+NoConn ~ 7050 6000
+NoConn ~ 7050 6100
+NoConn ~ 4100 6450
+NoConn ~ 12400 6850
+NoConn ~ 12400 7900
+Wire Wire Line
+	6750 5400 6750 5450
+NoConn ~ 8500 7250
+Wire Wire Line
+	5750 5650 5750 5700
+Connection ~ 5750 5700
+Connection ~ 12550 7100
+Text Label 6200 5250 0    50   ~ 0
+D+
+Text Label 6200 5350 0    50   ~ 0
+D-
 $EndSCHEMATC
