File: file59F1F748.sch (KiCad schematic (older format))
At the start: 51 parts, among them J3 BARREL_JACK, U10 L78L15_SO8, U11 L79L15_SO8, U12 TPS563209, U13 TPS563209, U7 LM27313, U8 LM43601, U9 L78L05_SO8

Commit message: Updated schematics and part number fields
Parts:
- D1: value D -> SK34ATR; footprint (none) -> Diodes_SMD:D_SMA_Handsoldering; mpn (none) -> SK34ATR
- D2: value D_Schottky -> SK34ATR; footprint (none) -> Diodes_SMD:D_SMA_Handsoldering; mpn (none) -> SK34ATR
- F1: footprint (none) -> Resistors_SMD:R_1812_HandSoldering; mpn (none) -> 0ZCG0200FF2C
- J3: footprint (none) -> Connectors:BARREL_JACK; mpn (none) -> PJ-037A
- L1: footprint (none) -> Inductors_SMD:L_7.3x7.3_H3.5; mpn (none) -> PA4332.103NLT
- L2: footprint (none) -> Inductors_SMD:L_12x12mm_h4.5mm; mpn (none) -> SDR1105-560KL
- L3, L4: footprint (none) -> Inductors_SMD:L_Taiyo-Yuden_NR-50xx_HandSoldering; mpn (none) -> NRS5012T2R2MMGF
- R13: value 13K7 -> 1K; MPN (none) -> RC0805FR-071KL
- R14: MPN (none) -> RC0805FR-0760K4L
- R16: MPN (none) -> RC0805FR-07187KL
- R17: MPN (none) -> RC0805FR-071ML
- R18: mpn (none) -> RC0805FR-0733K2L
- R19: MPN (none) -> RC0805FR-0710K2L
- R20: MPN (none) -> RC0805FR-073K74L
- R21: MPN (none) -> RC0805FR-0710KL
- U12, U13: footprint (none) -> TO_SOT_Packages_SMD:SOT-23-6_Handsoldering
- U7: footprint (none) -> TO_SOT_Packages_SMD:SOT-23-5_HandSoldering
- U8: footprint (none) -> Housings_SSOP:SSOP-16_4.4x5.2mm_Pitch0.65mm
Changed lines of the file:
@@
 F 0 "J3" H 1400 1495 50  0000 C CNN
 F 1 "BARREL_JACK" H 1400 1145 50  0000 C CNN
-F 2 "" H 1400 1300 50  0001 C CNN
+F 2 "Connectors:BARREL_JACK" H 1400 1300 50  0001 C CNN
 F 3 "" H 1400 1300 50  0001 C CNN
+F 4 "PJ-037A" H 1400 1300 60  0001 C CNN "mpn"
 	1    1400 1300
 	1    0    0    -1
 $EndComp
 $Comp
-L GND #PWR028
+L GND #PWR31
 U 1 1 59F1F7D5
 P 2250 1550
-F 0 "#PWR028" H 2250 1300 50  0001 C CNN
+F 0 "#PWR31" H 2250 1300 50  0001 C CNN
 F 1 "GND" H 2250 1400 50  0000 C CNN
 F 2 "" H 2250 1550 50  0001 C CNN
@@
 $EndComp
 $Comp
-L VCC #PWR029
+L VCC #PWR30
 U 1 1 59F1F7EB
 P 2250 1050
-F 0 "#PWR029" H 2250 900 50  0001 C CNN
+F 0 "#PWR30" H 2250 900 50  0001 C CNN
 F 1 "VCC" H 2250 1200 50  0000 C CNN
 F 2 "" H 2250 1050 50  0001 C CNN
@@
 	3650 3300 3650 3800
 $Comp
-L +15V #PWR030
+L +15V #PWR38
 U 1 1 59F1FEE5
 P 4450 3700
-F 0 "#PWR030" H 4450 3550 50  0001 C CNN
+F 0 "#PWR38" H 4450 3550 50  0001 C CNN
 F 1 "+15V" H 4450 3840 50  0000 C CNN
 F 2 "" H 4450 3700 50  0001 C CNN
@@
 $EndComp
 $Comp
-L -12VA #PWR031
+L -12VA #PWR39
 U 1 1 59F1FF38
 P 4450 4500
-F 0 "#PWR031" H 4450 4350 50  0001 C CNN
+F 0 "#PWR39" H 4450 4350 50  0001 C CNN
 F 1 "-12VA" H 4450 4640 50  0000 C CNN
 F 2 "" H 4450 4500 50  0001 C CNN
@@
 F 0 "U7" H 1750 3750 60  0000 C CNN
 F 1 "LM27313" H 1750 3650 60  0000 C CNN
-F 2 "" H 1750 3650 60  0001 C CNN
+F 2 "TO_SOT_Packages_SMD:SOT-23-5_HandSoldering" H 1750 3650 60  0001 C CNN
 F 3 "" H 1750 3650 60  0001 C CNN
 F 4 "LM27313XMF/NOPB" H 1750 3650 60  0001 C CNN "mpn"
@@
 F 0 "L1" V 1750 3300 50  0000 C CNN
 F 1 "10u" V 1875 3300 50  0000 C CNN
-F 2 "" H 1800 3300 50  0001 C CNN
+F 2 "Inductors_SMD:L_7.3x7.3_H3.5" H 1800 3300 50  0001 C CNN
 F 3 "" H 1800 3300 50  0001 C CNN
+F 4 "PA4332.103NLT" V 1800 3300 60  0001 C CNN "mpn"
 	1    1800 3300
 	0    -1   -1   0
@@
 P 2450 3300
 F 0 "D2" H 2450 3400 50  0000 C CNN
-F 1 "D_Schottky" H 2450 3200 50  0000 C CNN
-F 2 "" H 2450 3300 50  0001 C CNN
+F 1 "SK34ATR" H 2450 3200 50  0000 C CNN
+F 2 "Diodes_SMD:D_SMA_Handsoldering" H 2450 3300 50  0001 C CNN
 F 3 "" H 2450 3300 50  0001 C CNN
+F 4 "SK34ATR" H 2450 3300 60  0001 C CNN "mpn"
 	1    2450 3300
 	-1   0    0    1
@@
 F 2 "Resistors_SMD:R_0805_HandSoldering" V 2680 3450 50  0001 C CNN
 F 3 "" H 2750 3450 50  0001 C CNN
+F 4 "RC0805FR-07187KL" V 2750 3450 60  0001 C CNN "MPN"
 	1    2750 3450
 	1    0    0    -1
@@
 P 1250 3600
 F 0 "R13" V 1330 3600 50  0000 C CNN
-F 1 "13K7" V 1250 3600 50  0000 C CNN
+F 1 "1K" V 1250 3600 50  0000 C CNN
 F 2 "Resistors_SMD:R_0805_HandSoldering" V 1180 3600 50  0001 C CNN
 F 3 "" H 1250 3600 50  0001 C CNN
+F 4 "RC0805FR-071KL" V 1250 3600 60  0001 C CNN "MPN"
 	1    1250 3600
 	-1   0    0    1
@@
 Connection ~ 1400 3300
 $Comp
-L VCC #PWR032
+L VCC #PWR28
 U 1 1 5A046DAC
 P 1250 3250
-F 0 "#PWR032" H 1250 3100 50  0001 C CNN
+F 0 "#PWR28" H 1250 3100 50  0001 C CNN
 F 1 "VCC" H 1250 3400 50  0000 C CNN
 F 2 "" H 1250 3250 50  0001 C CNN
@@
 Connection ~ 1250 3300
 $Comp
-L GND #PWR033
+L GND #PWR32
 U 1 1 5A046E95
 P 2450 3900
-F 0 "#PWR033" H 2450 3650 50  0001 C CNN
+F 0 "#PWR32" H 2450 3650 50  0001 C CNN
 F 1 "GND" H 2450 3750 50  0000 C CNN
 F 2 "" H 2450 3900 50  0001 C CNN
@@
 F 0 "U8" H 2000 5150 60  0000 C CNN
 F 1 "LM43601" H 2000 5050 60  0000 C CNN
-F 2 "" H 2000 5050 60  0001 C CNN
+F 2 "Housings_SSOP:SSOP-16_4.4x5.2mm_Pitch0.65mm" H 2000 5050 60  0001 C CNN
 F 3 "" H 2000 5050 60  0001 C CNN
 F 4 "LM43601PWPR" H 2000 5050 60  0001 C CNN "mpn"
@@
 F 0 "L2" V 2900 5150 50  0000 C CNN
 F 1 "56u" V 3025 5150 50  0000 C CNN
-F 2 "" H 2950 5150 50  0001 C CNN
+F 2 "Inductors_SMD:L_12x12mm_h4.5mm" H 2950 5150 50  0001 C CNN
 F 3 "" H 2950 5150 50  0001 C CNN
+F 4 "SDR1105-560KL" V 2950 5150 60  0001 C CNN "mpn"
 	1    2950 5150
 	0    -1   -1   0
@@
 Connection ~ 2200 5550
 $Comp
-L VCC #PWR034
+L VCC #PWR29
 U 1 1 5A04B491
 P 2100 4600
-F 0 "#PWR034" H 2100 4450 50  0001 C CNN
+F 0 "#PWR29" H 2100 4450 50  0001 C CNN
 F 1 "VCC" H 2100 4750 50  0000 C CNN
 F 2 "" H 2100 4600 50  0001 C CNN
@@
 F 2 "Resistors_SMD:R_0805_HandSoldering" V 2880 5250 50  0001 C CNN
 F 3 "" H 2950 5250 50  0001 C CNN
+F 4 "RC0805FR-071ML" V 2950 5250 60  0001 C CNN "MPN"
 	1    2950 5250
 	0    1    1    0
@@
 F 2 "Resistors_SMD:R_0805_HandSoldering" V 2480 5400 50  0001 C CNN
 F 3 "" H 2550 5400 50  0001 C CNN
+F 4 "RC0805FR-0760K4L" V 2550 5400 60  0001 C CNN "MPN"
 	1    2550 5400
 	-1   0    0    1
@@
 	2800 5450 2800 5250
 $Comp
-L GND #PWR035
+L GND #PWR35
 U 1 1 5A04BF4B
 P 3350 4850
-F 0 "#PWR035" H 3350 4600 50  0001 C CNN
+F 0 "#PWR35" H 3350 4600 50  0001 C CNN
 F 1 "GND" H 3350 4700 50  0000 C CNN
 F 2 "" H 3350 4850 50  0001 C CNN
@@
 Connection ~ 4050 5350
 $Comp
-L VCC #PWR036
+L VCC #PWR37
 U 1 1 5A04C911
 P 4250 5100
-F 0 "#PWR036" H 4250 4950 50  0001 C CNN
+F 0 "#PWR37" H 4250 4950 50  0001 C CNN
 F 1 "VCC" H 4250 5250 50  0000 C CNN
 F 2 "" H 4250 5100 50  0001 C CNN
@@
 $EndComp
 $Comp
-L +5V #PWR037
+L +5V #PWR36
 U 1 1 5A050046
 P 3400 2300
-F 0 "#PWR037" H 3400 2150 50  0001 C CNN
+F 0 "#PWR36" H 3400 2150 50  0001 C CNN
 F 1 "+5V" H 3400 2440 50  0000 C CNN
 F 2 "" H 3400 2300 50  0001 C CNN
@@
 Connection ~ 3000 2650
 $Comp
-L GND #PWR038
+L GND #PWR34
 U 1 1 5A0503BD
 P 3000 2700
-F 0 "#PWR038" H 3000 2450 50  0001 C CNN
+F 0 "#PWR34" H 3000 2450 50  0001 C CNN
 F 1 "GND" H 3000 2550 50  0000 C CNN
 F 2 "" H 3000 2700 50  0001 C CNN
@@
 	3000 2700 3000 2650
 $Comp
-L VCC #PWR039
+L VCC #PWR33
 U 1 1 5A0504E4
 P 2700 2250
-F 0 "#PWR039" H 2700 2100 50  0001 C CNN
+F 0 "#PWR33" H 2700 2100 50  0001 C CNN
 F 1 "VCC" H 2700 2400 50  0000 C CNN
 F 2 "" H 2700 2250 50  0001 C CNN
@@
 F 0 "U12" H 5250 1850 60  0000 C CNN
 F 1 "TPS563209" H 5250 1750 60  0000 C CNN
-F 2 "" H 5250 1750 60  0001 C CNN
+F 2 "TO_SOT_Packages_SMD:SOT-23-6_Handsoldering" H 5250 1750 60  0001 C CNN
 F 3 "" H 5250 1750 60  0001 C CNN
 F 4 "TPS563209DDCT" H 5250 1750 60  0001 C CNN "mpn"
@@
 F 0 "L3" V 5950 1650 50  0000 C CNN
 F 1 "2u2" V 6075 1650 50  0000 C CNN
-F 2 "" H 6000 1650 50  0001 C CNN
+F 2 "Inductors_SMD:L_Taiyo-Yuden_NR-50xx_HandSoldering" H 6000 1650 50  0001 C CNN
 F 3 "" H 6000 1650 50  0001 C CNN
+F 4 "NRS5012T2R2MMGF" V 6000 1650 60  0001 C CNN "mpn"
 	1    6000 1650
 	0    -1   -1   0
@@
 F 2 "Resistors_SMD:R_0805_HandSoldering" V 5930 1800 50  0001 C CNN
 F 3 "" H 6000 1800 50  0001 C CNN
+F 4 "RC0805FR-0733K2L" V 6000 1800 60  0001 C CNN "mpn"
 	1    6000 1800
 	0    -1   -1   0
@@
 F 2 "Resistors_SMD:R_0805_HandSoldering" V 5930 1900 50  0001 C CNN
 F 3 "" H 6000 1900 50  0001 C CNN
+F 4 "RC0805FR-0710K2L" V 6000 1900 60  0001 C CNN "MPN"
 	1    6000 1900
 	0    1    1    0
@@
 	4900 1500 4900 1650
 $Comp
-L VCC #PWR040
+L VCC #PWR40
 U 1 1 5A052B3C
 P 4900 1500
-F 0 "#PWR040" H 4900 1350 50  0001 C CNN
+F 0 "#PWR40" H 4900 1350 50  0001 C CNN
 F 1 "VCC" H 4900 1650 50  0000 C CNN
 F 2 "" H 4900 1500 50  0001 C CNN
@@
 Connection ~ 4900 1550
 $Comp
-L +3V3 #PWR041
+L +3V3 #PWR41
 U 1 1 5A052CCD
 P 6700 1600
-F 0 "#PWR041" H 6700 1450 50  0001 C CNN
+F 0 "#PWR41" H 6700 1450 50  0001 C CNN
 F 1 "+3V3" H 6700 1740 50  0000 C CNN
 F 2 "" H 6700 1600 50  0001 C CNN
@@
 F 0 "U13" H 7900 1900 60  0000 C CNN
 F 1 "TPS563209" H 7900 1800 60  0000 C CNN
-F 2 "" H 7900 1800 60  0001 C CNN
+F 2 "TO_SOT_Packages_SMD:SOT-23-6_Handsoldering" H 7900 1800 60  0001 C CNN
 F 3 "" H 7900 1800 60  0001 C CNN
 	1    7900 1800
@@
 F 0 "L4" V 8600 1700 50  0000 C CNN
 F 1 "2u2" V 8725 1700 50  0000 C CNN
-F 2 "" H 8650 1700 50  0001 C CNN
+F 2 "Inductors_SMD:L_Taiyo-Yuden_NR-50xx_HandSoldering" H 8650 1700 50  0001 C CNN
 F 3 "" H 8650 1700 50  0001 C CNN
+F 4 "NRS5012T2R2MMGF" V 8650 1700 60  0001 C CNN "mpn"
 	1    8650 1700
 	0    -1   -1   0
@@
 F 2 "Resistors_SMD:R_0805_HandSoldering" V 8580 1850 50  0001 C CNN
 F 3 "" H 8650 1850 50  0001 C CNN
+F 4 "RC0805FR-073K74L" V 8650 1850 60  0001 C CNN "MPN"
 	1    8650 1850
 	0    -1   -1   0
@@
 F 2 "Resistors_SMD:R_0805_HandSoldering" V 8580 1950 50  0001 C CNN
 F 3 "" H 8650 1950 50  0001 C CNN
+F 4 "RC0805FR-0710KL" V 8650 1950 60  0001 C CNN "MPN"
 	1    8650 1950
 	0    1    1    0
@@
 Connection ~ 8500 1900
 $Comp
-L VCC #PWR042
+L VCC #PWR42
 U 1 1 5A053577
 P 7550 1550
-F 0 "#PWR042" H 7550 1400 50  0001 C CNN
+F 0 "#PWR42" H 7550 1400 50  0001 C CNN
 F 1 "VCC" H 7550 1700 50  0000 C CNN
 F 2 "" H 7550 1550 50  0001 C CNN
@@
 Connection ~ 6700 1650
 $Comp
-L +1V0 #PWR043
+L +1V0 #PWR43
 U 1 1 5A0539BE
 P 9350 1650
-F 0 "#PWR043" H 9350 1500 50  0001 C CNN
+F 0 "#PWR43" H 9350 1500 50  0001 C CNN
 F 1 "+1V0" H 9350 1790 50  0000 C CNN
 F 2 "" H 9350 1650 50  0001 C CNN
@@
 F 0 "F1" V 1775 1200 50  0000 C CNN
 F 1 "2A" V 1925 1200 50  0000 C CNN
-F 2 "" H 1900 1000 50  0001 L CNN
+F 2 "Resistors_SMD:R_1812_HandSoldering" H 1900 1000 50  0001 L CNN
 F 3 "" H 1850 1200 50  0001 C CNN
+F 4 "0ZCG0200FF2C" V 1850 1200 60  0001 C CNN "mpn"
 	1    1850 1200
 	0    1    1    0
@@
 P 2050 1350
 F 0 "D1" H 2050 1450 50  0000 C CNN
-F 1 "D" H 2050 1250 50  0000 C CNN
-F 2 "" H 2050 1350 50  0001 C CNN
+F 1 "SK34ATR" H 2050 1250 50  0000 C CNN
+F 2 "Diodes_SMD:D_SMA_Handsoldering" H 2050 1350 50  0001 C CNN
 F 3 "" H 2050 1350 50  0001 C CNN
+F 4 "SK34ATR" H 2050 1350 60  0001 C CNN "mpn"
 	1    2050 1350
 	0    1    1    0

Commit message: Began PCB layout
Parts:
- removed C28: 120p, Capacitors_SMD:C_0805_HandSoldering, symbol C_Small
- removed C29, C30, C38: 4u7, Capacitors_SMD:C_0805_HandSoldering, symbol C_Small
- removed C32, C35, C36, C37: 10u, Capacitors_SMD:C_0805_HandSoldering, symbol C_Small
- removed D2: SK34ATR, Diodes_SMD:D_SMA_Handsoldering, symbol D_Schottky
- removed F1: 2A, Resistors_SMD:R_1812_HandSoldering, symbol Polyfuse_Small
- removed L1: 10u, Inductors_SMD:L_7.3x7.3_H3.5, symbol L
- removed L2: 56u, Inductors_SMD:L_12x12mm_h4.5mm, symbol L
- removed R13: 1K, Resistors_SMD:R_0805_HandSoldering, symbol R
- removed R14: 60K4, Resistors_SMD:R_0805_HandSoldering, symbol R
- removed R15: 13K7, Resistors_SMD:R_0805_HandSoldering, symbol R
- removed R16: 187K, Resistors_SMD:R_0805_HandSoldering, symbol R
- removed R17: 1M, Resistors_SMD:R_0805_HandSoldering, symbol R
- removed U10: L78L15_SO8, Housings_SOIC:SOIC-8_3.9x4.9mm_Pitch1.27mm, symbol L78L15_SO8
- removed U11: L79L15_SO8, Housings_SOIC:SOIC-8_3.9x4.9mm_Pitch1.27mm, symbol L79L15_SO8
- removed U7: LM27313, TO_SOT_Packages_SMD:SOT-23-5_HandSoldering, symbol LM27313
- removed U8: LM43601, Housings_SSOP:SSOP-16_4.4x5.2mm_Pitch0.65mm, symbol LM43601
- added C1: 100n, Capacitors_SMD:C_0805_HandSoldering, symbol C_Small
- added U10: L79L12_SO8, Housings_SOIC:SOIC-8_3.9x4.9mm_Pitch1.27mm, symbol L79L12_SO8
- added U11: AP1117-33, TO_SOT_Packages_SMD:SOT-223-3_TabPin2, symbol AP1117-33
- added U7: CHINADCDC, dacparts:chinadcdc, symbol CHINADCDC
- added U8: LM78L12_SO8, Housings_SOIC:SOIC-8_3.9x4.9mm_Pitch1.27mm, symbol LM78L12_SO8
- C22: value 2u2 -> 22u; mpn CL21A225KAFNNNG -> (none)
- C24: value 470n -> 22u; mpn CL21F473ZBANNNC -> (none)
- C27: value 110p -> 100n
- D1: mpn SK34ATR -> SS210ATR
Connections:
- net labels added: +12V, +3.3VA, -12V, GNDD, VBUS
- net labels removed: +15V, +18V, -12VA, -18V
- wire segments 112 -> 83
- no-connect marks 4 -> 0
Other:
- note added: "12/-12v Analog supply\n100mA max"
- note removed: "-18v Inverter"
- note removed: "15/-15v Analog supply\n100mA max"
- note removed: "18v Boost Converter"
- moved on the sheet: D1

Commit message: updated to new kicad format
Parts:
- C1, C22, C24, C25, C26, C27, C31, C33, C34, C39, C40, C41, C42, C43, C44, C45, C46, C47, C48: symbol C_Small -> Device:C_Small
- C23: symbol CP1_Small -> Device:CP1_Small
- D1: symbol D -> Device:D
- J3: symbol BARREL_JACK -> Connector_Specialized:Barrel_Jack
- L3, L4: symbol L -> Device:L
- R18, R19, R20, R21: symbol R -> Device:R
- U10: symbol L79L12_SO8 -> Regulator_Linear:L79L12_SO8
- U11: symbol AP1117-33 -> Regulator_Linear:AP1117-33
- U12, U13: symbol TPS563209 -> dacparts:TPS563209
- U7: symbol CHINADCDC -> dacparts:CHINADCDC
- U8: symbol LM78L12_SO8 -> Regulator_Linear:LM78L12_SO8
- U9: symbol L78L05_SO8 -> Regulator_Linear:L78L05_SO8
Connections:
- wire segments 83 -> 120
Other:
- note added: "3.3V DAC Digital supply"
- note added: "USB Supply (Isolated)"
- moved on the sheet: C1, C22, C24, C25, C27, C31, C33, C34, C39, C40, C41, C42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

Commit message: started routing PCB
Parts:
- C1, C25, C26, C27, C31, C33, C34, C39, C40: footprint Capacitors_SMD:C_0805_HandSoldering -> Capacitors_SMD:C_0402
- C22, C24, C41, C42, C45, C46: footprint Capacitors_SMD:C_0805_HandSoldering -> Capacitors_SMD:C_0805
- C43, C44, C47, C48: footprint Capacitors_SMD:C_0805_HandSoldering -> Capacitors_SMD:C_1206
- R18, R19, R20, R21: footprint Resistors_SMD:R_0805_HandSoldering -> Resistors_SMD:R_0402
Connections:
- wire segments 120 -> 119
Changed lines of the file:
@@
 EESchema Schematic File Version 4
+LIBS:USB-DAC-cache
 EELAYER 26 0
 EELAYER END
@@
 F 0 "C26" H 2760 1370 50  0000 L CNN
 F 1 "100n" H 2750 1150 50  0000 L CNN
-F 2 "Capacitors_SMD:C_0805_HandSoldering" H 2750 1300 50  0001 C CNN
+F 2 "Capacitors_SMD:C_0402" H 2750 1300 50  0001 C CNN
 F 3 "" H 2750 1300 50  0001 C CNN
 	1    2750 1300
@@
 F 0 "C39" H 3260 2570 50  0000 L CNN
 F 1 "100n" H 3250 2350 50  0000 L CNN
-F 2 "Capacitors_SMD:C_0805_HandSoldering" H 3250 2500 50  0001 C CNN
+F 2 "Capacitors_SMD:C_0402" H 3250 2500 50  0001 C CNN
 F 3 "" H 3250 2500 50  0001 C CNN
 	1    3250 2500
@@
 F 0 "C40" H 3260 2970 50  0000 L CNN
 F 1 "100n" H 3250 2750 50  0000 L CNN
-F 2 "Capacitors_SMD:C_0805_HandSoldering" H 3250 2900 50  0001 C CNN
+F 2 "Capacitors_SMD:C_0402" H 3250 2900 50  0001 C CNN
 F 3 "" H 3250 2900 50  0001 C CNN
 	1    3250 2900
@@
 F 0 "C33" H 2460 2570 50  0000 L CNN
 F 1 "100n" H 2450 2350 50  0000 L CNN
-F 2 "Capacitors_SMD:C_0805_HandSoldering" H 2450 2500 50  0001 C CNN
+F 2 "Capacitors_SMD:C_0402" H 2450 2500 50  0001 C CNN
 F 3 "" H 2450 2500 50  0001 C CNN
 	1    2450 2500
@@
 F 0 "C34" H 2460 2920 50  0000 L CNN
 F 1 "100n" H 2450 2700 50  0000 L CNN
-F 2 "Capacitors_SMD:C_0805_HandSoldering" H 2450 2850 50  0001 C CNN
+F 2 "Capacitors_SMD:C_0402" H 2450 2850 50  0001 C CNN
 F 3 "" H 2450 2850 50  0001 C CNN
 	1    2450 2850
@@
 F 0 "C31" H 1760 4370 50  0000 L CNN
 F 1 "100n" H 1750 4150 50  0000 L CNN
-F 2 "Capacitors_SMD:C_0805_HandSoldering" H 1750 4300 50  0001 C CNN
+F 2 "Capacitors_SMD:C_0402" H 1750 4300 50  0001 C CNN
 F 3 "" H 1750 4300 50  0001 C CNN
 	1    1750 4300
@@
 F 0 "C25" H 1160 4370 50  0000 L CNN
 F 1 "100n" H 1150 4150 50  0000 L CNN
-F 2 "Capacitors_SMD:C_0805_HandSoldering" H 1150 4300 50  0001 C CNN
+F 2 "Capacitors_SMD:C_0402" H 1150 4300 50  0001 C CNN
 F 3 "" H 1150 4300 50  0001 C CNN
 	1    1150 4300
@@
 F 0 "C41" H 5760 1570 50  0000 L CNN
 F 1 "100n" H 5760 1420 50  0000 L CNN
-F 2 "Capacitors_SMD:C_0805_HandSoldering" H 5750 1500 50  0001 C CNN
+F 2 "Capacitors_SMD:C_0805" H 5750 1500 50  0001 C CNN
 F 3 "" H 5750 1500 50  0001 C CNN
 	1    5750 1500
@@
 F 0 "C43" H 6510 1770 50  0000 L CNN
 F 1 "47u" H 6510 1620 50  0000 L CNN
-F 2 "Capacitors_SMD:C_0805_HandSoldering" H 6500 1700 50  0001 C CNN
+F 2 "Capacitors_SMD:C_1206" H 6500 1700 50  0001 C CNN
 F 3 "" H 6500 1700 50  0001 C CNN
 F 4 "CL21A476MQYNNNE" H 6500 1700 60  0001 C CNN "mpn"
@@
 F 0 "C44" H 6710 1770 50  0000 L CNN
 F 1 "47u" H 6710 1620 50  0000 L CNN
-F 2 "Capacitors_SMD:C_0805_HandSoldering" H 6700 1700 50  0001 C CNN
+F 2 "Capacitors_SMD:C_1206" H 6700 1700 50  0001 C CNN
 F 3 "" H 6700 1700 50  0001 C CNN
 	1    6700 1700
@@
 F 0 "C42" H 6260 1770 50  0000 L CNN
 F 1 "100n" H 6260 1620 50  0000 L CNN
-F 2 "Capacitors_SMD:C_0805_HandSoldering" H 6250 1700 50  0001 C CNN
+F 2 "Capacitors_SMD:C_0805" H 6250 1700 50  0001 C CNN
 F 3 "" H 6250 1700 50  0001 C CNN
 	1    6250 1700
@@
 F 0 "R18" V 6080 1750 50  0000 C CNN
 F 1 "33K2" V 6000 1750 50  0000 C CNN
-F 2 "Resistors_SMD:R_0805_HandSoldering" V 5930 1750 50  0001 C CNN
+F 2 "Resistors_SMD:R_0402" V 5930 1750 50  0001 C CNN
 F 3 "" H 6000 1750 50  0001 C CNN
 F 4 "RC0805FR-0733K2L" V 6000 1750 60  0001 C CNN "mpn"
@@
 F 0 "R19" V 6080 1850 50  0000 C CNN
 F 1 "10K2" V 6000 1850 50  0000 C CNN
-F 2 "Resistors_SMD:R_0805_HandSoldering" V 5930 1850 50  0001 C CNN
+F 2 "Resistors_SMD:R_0402" V 5930 1850 50  0001 C CNN
 F 3 "" H 6000 1850 50  0001 C CNN
 F 4 "RC0805FR-0710K2L" V 6000 1850 60  0001 C CNN "MPN"
@@
 F 0 "C45" H 8410 1670 50  0000 L CNN
 F 1 "100n" H 8410 1520 50  0000 L CNN
-F 2 "Capacitors_SMD:C_0805_HandSoldering" H 8400 1600 50  0001 C CNN
+F 2 "Capacitors_SMD:C_0805" H 8400 1600 50  0001 C CNN
 F 3 "" H 8400 1600 50  0001 C CNN
 	1    8400 1600
@@
 F 0 "C47" H 9160 1870 50  0000 L CNN
 F 1 "47u" H 9160 1720 50  0000 L CNN
-F 2 "Capacitors_SMD:C_0805_HandSoldering" H 9150 1800 50  0001 C CNN
+F 2 "Capacitors_SMD:C_1206" H 9150 1800 50  0001 C CNN
 F 3 "" H 9150 1800 50  0001 C CNN
 	1    9150 1800
@@
 F 0 "C48" H 9360 1870 50  0000 L CNN
 F 1 "47u" H 9360 1720 50  0000 L CNN
-F 2 "Capacitors_SMD:C_0805_HandSoldering" H 9350 1800 50  0001 C CNN
+F 2 "Capacitors_SMD:C_1206" H 9350 1800 50  0001 C CNN
 F 3 "" H 9350 1800 50  0001 C CNN
 	1    9350 1800
@@
 F 0 "C46" H 8910 1870 50  0000 L CNN
 F 1 "100n" H 8910 1720 50  0000 L CNN
-F 2 "Capacitors_SMD:C_0805_HandSoldering" H 8900 1800 50  0001 C CNN
+F 2 "Capacitors_SMD:C_0805" H 8900 1800 50  0001 C CNN
 F 3 "" H 8900 1800 50  0001 C CNN
 	1    8900 1800
@@
 F 0 "R20" V 8730 1850 50  0000 C CNN
 F 1 "3K74" V 8650 1850 50  0000 C CNN
-F 2 "Resistors_SMD:R_0805_HandSoldering" V 8580 1850 50  0001 C CNN
+F 2 "Resistors_SMD:R_0402" V 8580 1850 50  0001 C CNN
 F 3 "" H 8650 1850 50  0001 C CNN
 F 4 "RC0805FR-073K74L" V 8650 1850 60  0001 C CNN "MPN"
@@
 F 0 "R21" V 8730 1950 50  0000 C CNN
 F 1 "10K" V 8650 1950 50  0000 C CNN
-F 2 "Resistors_SMD:R_0805_HandSoldering" V 8580 1950 50  0001 C CNN
+F 2 "Resistors_SMD:R_0402" V 8580 1950 50  0001 C CNN
 F 3 "" H 8650 1950 50  0001 C CNN
 F 4 "RC0805FR-0710KL" V 8650 1950 60  0001 C CNN "MPN"
@@
 	1    0    0    -1
 $EndComp
-Wire Wire Line
-	7350 1600 7550 1600
 Wire Wire Line
 	7400 1750 7550 1750
@@
 F 0 "C22" H 2260 2570 50  0000 L CNN
 F 1 "22u" H 2250 2350 50  0000 L CNN
-F 2 "Capacitors_SMD:C_0805_HandSoldering" H 2250 2500 50  0001 C CNN
+F 2 "Capacitors_SMD:C_0805" H 2250 2500 50  0001 C CNN
 F 3 "" H 2250 2500 50  0001 C CNN
 	1    2250 2500
@@
 F 0 "C24" H 2260 2920 50  0000 L CNN
 F 1 "22u" H 2250 2700 50  0000 L CNN
-F 2 "Capacitors_SMD:C_0805_HandSoldering" H 2250 2850 50  0001 C CNN
+F 2 "Capacitors_SMD:C_0805" H 2250 2850 50  0001 C CNN
 F 3 "" H 2250 2850 50  0001 C CNN
 	1    2250 2850
@@
 P 5550 2000
 F 0 "#PWR015" H 5550 1750 50  0001 C CNN
-F 1 "GNDD" H 5550 1875 50  0000 C CNN
+F 1 "GNDD" H 5800 1950 50  0000 C CNN
 F 2 "" H 5550 2000 50  0001 C CNN
 F 3 "" H 5550 2000 50  0001 C CNN
@@
 F 0 "C1" H 2260 4370 50  0000 L CNN
 F 1 "100n" H 2250 4150 50  0000 L CNN
-F 2 "Capacitors_SMD:C_0805_HandSoldering" H 2250 4300 50  0001 C CNN
+F 2 "Capacitors_SMD:C_0402" H 2250 4300 50  0001 C CNN
 F 3 "" H 2250 4300 50  0001 C CNN
 	1    2250 4300
@@
 F 0 "C27" H 2860 4370 50  0000 L CNN
 F 1 "100n" H 2850 4150 50  0000 L CNN
-F 2 "Capacitors_SMD:C_0805_HandSoldering" H 2850 4300 50  0001 C CNN
+F 2 "Capacitors_SMD:C_0402" H 2850 4300 50  0001 C CNN
 F 3 "" H 2850 4300 50  0001 C CNN
 	1    2850 4300
@@
 Wire Wire Line
 	8500 1900 8500 1950
-Wire Wire Line
-	6700 1600 7350 1600
 Wire Wire Line
 	2450 1550 2750 1550
@@
 Connection ~ 5850 1600
 Connection ~ 6150 1600
+Wire Wire Line
+	6700 1600 7550 1600
 $EndSCHEMATC
