File: file5A0DCEA9.sch (KiCad schematic (older format))
At the start: 8 parts, among them J4 XLR3, J5 XLR3, U17 DRV135, U18 DRV135

Commit message: Updated schematics and part number fields
Parts:
- removed J4, J5: XLR3, symbol XLR3
- added J4, J5: JACK_TRS_6PINS, symbol JACK_TRS_6PINS
Connections:
- wire segments 36 -> 39
Changed lines of the file:
@@
-$EndComp
-$Comp
-L XLR3 J4
-U 1 1 5A0DE654
-P 6550 2200
-F 0 "J4" H 6700 2450 50  0000 C CNN
-F 1 "XLR3" H 6750 1950 50  0000 C CNN
-F 2 "" H 6550 2200 50  0001 C CNN
-F 3 "" H 6550 2200 50  0001 C CNN
-	1    6550 2200
-	1    0    0    -1
 $EndComp
 $Comp
@@
 	5950 2300 5950 2400
 $Comp
-L GND #PWR065
+L GND #PWR65
 U 1 1 5A0DE91C
 P 4450 2350
-F 0 "#PWR065" H 4450 2100 50  0001 C CNN
+F 0 "#PWR65" H 4450 2100 50  0001 C CNN
 F 1 "GND" H 4450 2200 50  0000 C CNN
 F 2 "" H 4450 2350 50  0001 C CNN
@@
 Connection ~ 4750 2300
 $Comp
-L +15V #PWR066
+L +15V #PWR67
 U 1 1 5A0DE955
 P 5000 1850
-F 0 "#PWR066" H 5000 1700 50  0001 C CNN
+F 0 "#PWR67" H 5000 1700 50  0001 C CNN
 F 1 "+15V" H 5000 1990 50  0000 C CNN
 F 2 "" H 5000 1850 50  0001 C CNN
@@
 $EndComp
 $Comp
-L -12VA #PWR067
+L -12VA #PWR68
 U 1 1 5A0DE975
 P 5000 2550
-F 0 "#PWR067" H 5000 2400 50  0001 C CNN
+F 0 "#PWR68" H 5000 2400 50  0001 C CNN
 F 1 "-12VA" H 5000 2690 50  0000 C CNN
 F 2 "" H 5000 2550 50  0001 C CNN
@@
 Connection ~ 5000 1900
 Wire Wire Line
-	5950 2400 6400 2400
-Wire Wire Line
-	6400 2400 6400 2550
-Wire Wire Line
-	6400 2550 6550 2550
-Wire Wire Line
-	5950 2100 6150 2100
-Wire Wire Line
-	6150 2100 6150 1950
-Wire Wire Line
-	6150 1950 6900 1950
-Wire Wire Line
-	6900 1950 6900 2200
-$Comp
-L GND #PWR068
-U 1 1 5A0DEA54
-P 6150 2200
-F 0 "#PWR068" H 6150 1950 50  0001 C CNN
-F 1 "GND" H 6150 2050 50  0000 C CNN
-F 2 "" H 6150 2200 50  0001 C CNN
-F 3 "" H 6150 2200 50  0001 C CNN
-	1    6150 2200
-	1    0    0    -1
-$EndComp
-Wire Wire Line
-	6150 2200 6200 2200
+	5950 2400 6550 2400
+Wire Wire Line
+	5950 2100 6350 2100
 $Comp
 L DRV135 U18
@@
 $EndComp
 $Comp
-L XLR3 J5
-U 1 1 5A0DEC46
-P 6550 3400
-F 0 "J5" H 6700 3650 50  0000 C CNN
-F 1 "XLR3" H 6750 3150 50  0000 C CNN
-F 2 "" H 6550 3400 50  0001 C CNN
-F 3 "" H 6550 3400 50  0001 C CNN
-	1    6550 3400
-	1    0    0    -1
-$EndComp
-$Comp
 L C_Small C65
 U 1 1 5A0DEC4C
@@
 	5950 3500 5950 3600
 $Comp
-L GND #PWR069
+L GND #PWR66
 U 1 1 5A0DEC62
 P 4450 3550
-F 0 "#PWR069" H 4450 3300 50  0001 C CNN
+F 0 "#PWR66" H 4450 3300 50  0001 C CNN
 F 1 "GND" H 4450 3400 50  0000 C CNN
 F 2 "" H 4450 3550 50  0001 C CNN
@@
 Connection ~ 4750 3500
 $Comp
-L +15V #PWR070
+L +15V #PWR69
 U 1 1 5A0DEC6A
 P 5000 3050
-F 0 "#PWR070" H 5000 2900 50  0001 C CNN
+F 0 "#PWR69" H 5000 2900 50  0001 C CNN
 F 1 "+15V" H 5000 3190 50  0000 C CNN
 F 2 "" H 5000 3050 50  0001 C CNN
@@
 $EndComp
 $Comp
-L -12VA #PWR071
+L -12VA #PWR70
 U 1 1 5A0DEC70
 P 5000 3750
-F 0 "#PWR071" H 5000 3600 50  0001 C CNN
+F 0 "#PWR70" H 5000 3600 50  0001 C CNN
 F 1 "-12VA" H 5000 3890 50  0000 C CNN
 F 2 "" H 5000 3750 50  0001 C CNN
@@
 	5950 3600 6400 3600
 Wire Wire Line
-	6400 3600 6400 3750
-Wire Wire Line
-	6400 3750 6550 3750
-Wire Wire Line
 	5950 3300 6150 3300
-Wire Wire Line
-	6150 3300 6150 3150
-Wire Wire Line
-	6150 3150 6900 3150
-Wire Wire Line
-	6900 3150 6900 3400
-$Comp
-L GND #PWR072
-U 1 1 5A0DEC7F
-P 6150 3400
-F 0 "#PWR072" H 6150 3150 50  0001 C CNN
-F 1 "GND" H 6150 3250 50  0000 C CNN
-F 2 "" H 6150 3400 50  0001 C CNN
-F 3 "" H 6150 3400 50  0001 C CNN
-	1    6150 3400
-	1    0    0    -1
-$EndComp
-Wire Wire Line
-	6150 3400 6200 3400
+$Comp
+L JACK_TRS_6PINS J5
+U 1 1 5A340C41
+P 7150 2300
+AR Path="/5A0DCEAA/5A340C41" Ref="J5"  Part="1"
+AR Path="/59E908E3/5A340C41" Ref="J5"  Part="1"
+F 0 "J5" H 7150 2700 50  0000 C CNN
+F 1 "JACK_TRS_6PINS" H 7100 2000 50  0000 C CNN
+F 2 "" H 7250 2150 50  0001 C CNN
+F 3 "" H 7250 2150 50  0001 C CNN
+F 4 "ACJS-MHOM" H 7150 2300 60  0001 C CNN "mpn"
+	1    7150 2300
+	-1   0    0    1
+$EndComp
+$Comp
+L JACK_TRS_6PINS J4
+U 1 1 5A340CC5
+P 7050 3500
+F 0 "J4" H 7050 3900 50  0000 C CNN
+F 1 "JACK_TRS_6PINS" H 7000 3200 50  0000 C CNN
+F 2 "" H 7150 3350 50  0001 C CNN
+F 3 "" H 7150 3350 50  0001 C CNN
+F 4 "ACJS-MHOM" H 7050 3500 60  0001 C CNN "mpn"
+	1    7050 3500
+	-1   0    0    1
+$EndComp
+$Comp
+L GND #PWR71
+U 1 1 5A340D6C
+P 6550 2550
+F 0 "#PWR71" H 6550 2300 50  0001 C CNN
+F 1 "GND" H 6550 2400 50  0000 C CNN
+F 2 "" H 6550 2550 50  0001 C CNN
+F 3 "" H 6550 2550 50  0001 C CNN
+	1    6550 2550
+	1    0    0    -1
+$EndComp
+Wire Wire Line
+	6550 2550 6550 2500
+Wire Wire Line
+	6550 2500 6750 2500
+Wire Wire Line
+	6750 2600 6700 2600
+Wire Wire Line
+	6700 2600 6700 2500
+Connection ~ 6700 2500
+$Comp
+L GND #PWR72
+U 1 1 5A340E0A
+P 6600 3850
+F 0 "#PWR72" H 6600 3600 50  0001 C CNN
+F 1 "GND" H 6600 3700 50  0000 C CNN
+F 2 "" H 6600 3850 50  0001 C CNN
+F 3 "" H 6600 3850 50  0001 C CNN
+	1    6600 3850
+	1    0    0    -1
+$EndComp
+Wire Wire Line
+	6600 3850 6600 3700
+Wire Wire Line
+	6600 3700 6650 3700
+Wire Wire Line
+	6650 3800 6600 3800
+Connection ~ 6600 3800
+Wire Wire Line
+	6650 3500 6150 3500
+Wire Wire Line
+	6150 3500 6150 3300
+Wire Wire Line
+	6400 3600 6400 3300
+Wire Wire Line
+	6400 3300 6650 3300
+Wire Wire Line
+	6750 2300 6350 2300
+Wire Wire Line
+	6350 2300 6350 2100
+Wire Wire Line
+	6550 2400 6550 2100
+Wire Wire Line
+	6550 2100 6750 2100
 $EndSCHEMATC

Commit message: Began PCB layout
Parts:
- C63, C64, C65, C66: value 0.1u -> 100n
- J4, J5: footprint (none) -> Connectors:NMJ6HCD2
Changed lines of the file:
@@
 P 4750 2000
 F 0 "C63" H 4760 2070 50  0000 L CNN
-F 1 "0.1u" H 4760 1920 50  0000 L CNN
+F 1 "100n" H 4760 1920 50  0000 L CNN
 F 2 "Capacitors_SMD:C_0805_HandSoldering" H 4750 2000 50  0001 C CNN
 F 3 "" H 4750 2000 50  0001 C CNN
@@
 P 4750 2400
 F 0 "C64" H 4760 2470 50  0000 L CNN
-F 1 "0.1u" H 4760 2320 50  0000 L CNN
+F 1 "100n" H 4760 2320 50  0000 L CNN
 F 2 "Capacitors_SMD:C_0805_HandSoldering" H 4750 2400 50  0001 C CNN
 F 3 "" H 4750 2400 50  0001 C CNN
@@
 	5950 2300 5950 2400
 $Comp
-L GND #PWR65
+L GND #PWR041
 U 1 1 5A0DE91C
 P 4450 2350
-F 0 "#PWR65" H 4450 2100 50  0001 C CNN
+F 0 "#PWR041" H 4450 2100 50  0001 C CNN
 F 1 "GND" H 4450 2200 50  0000 C CNN
 F 2 "" H 4450 2350 50  0001 C CNN
@@
 Connection ~ 4750 2300
 $Comp
-L +15V #PWR67
+L +15V #PWR042
 U 1 1 5A0DE955
 P 5000 1850
-F 0 "#PWR67" H 5000 1700 50  0001 C CNN
+F 0 "#PWR042" H 5000 1700 50  0001 C CNN
 F 1 "+15V" H 5000 1990 50  0000 C CNN
 F 2 "" H 5000 1850 50  0001 C CNN
@@
 $EndComp
 $Comp
-L -12VA #PWR68
+L -12VA #PWR043
 U 1 1 5A0DE975
 P 5000 2550
-F 0 "#PWR68" H 5000 2400 50  0001 C CNN
+F 0 "#PWR043" H 5000 2400 50  0001 C CNN
 F 1 "-12VA" H 5000 2690 50  0000 C CNN
 F 2 "" H 5000 2550 50  0001 C CNN
@@
 P 4750 3200
 F 0 "C65" H 4760 3270 50  0000 L CNN
-F 1 "0.1u" H 4760 3120 50  0000 L CNN
+F 1 "100n" H 4760 3120 50  0000 L CNN
 F 2 "Capacitors_SMD:C_0805_HandSoldering" H 4750 3200 50  0001 C CNN
 F 3 "" H 4750 3200 50  0001 C CNN
@@
 P 4750 3600
 F 0 "C66" H 4760 3670 50  0000 L CNN
-F 1 "0.1u" H 4760 3520 50  0000 L CNN
+F 1 "100n" H 4760 3520 50  0000 L CNN
 F 2 "Capacitors_SMD:C_0805_HandSoldering" H 4750 3600 50  0001 C CNN
 F 3 "" H 4750 3600 50  0001 C CNN
@@
 	5950 3500 5950 3600
 $Comp
-L GND #PWR66
+L GND #PWR044
 U 1 1 5A0DEC62
 P 4450 3550
-F 0 "#PWR66" H 4450 3300 50  0001 C CNN
+F 0 "#PWR044" H 4450 3300 50  0001 C CNN
 F 1 "GND" H 4450 3400 50  0000 C CNN
 F 2 "" H 4450 3550 50  0001 C CNN
@@
 Connection ~ 4750 3500
 $Comp
-L +15V #PWR69
+L +15V #PWR045
 U 1 1 5A0DEC6A
 P 5000 3050
-F 0 "#PWR69" H 5000 2900 50  0001 C CNN
+F 0 "#PWR045" H 5000 2900 50  0001 C CNN
 F 1 "+15V" H 5000 3190 50  0000 C CNN
 F 2 "" H 5000 3050 50  0001 C CNN
@@
 $EndComp
 $Comp
-L -12VA #PWR70
+L -12VA #PWR046
 U 1 1 5A0DEC70
 P 5000 3750
-F 0 "#PWR70" H 5000 3600 50  0001 C CNN
+F 0 "#PWR046" H 5000 3600 50  0001 C CNN
 F 1 "-12VA" H 5000 3890 50  0000 C CNN
 F 2 "" H 5000 3750 50  0001 C CNN
@@
 F 0 "J5" H 7150 2700 50  0000 C CNN
 F 1 "JACK_TRS_6PINS" H 7100 2000 50  0000 C CNN
-F 2 "" H 7250 2150 50  0001 C CNN
+F 2 "Connectors:NMJ6HCD2" H 7250 2150 50  0001 C CNN
 F 3 "" H 7250 2150 50  0001 C CNN
 F 4 "ACJS-MHOM" H 7150 2300 60  0001 C CNN "mpn"
@@
 F 0 "J4" H 7050 3900 50  0000 C CNN
 F 1 "JACK_TRS_6PINS" H 7000 3200 50  0000 C CNN
-F 2 "" H 7150 3350 50  0001 C CNN
+F 2 "Connectors:NMJ6HCD2" H 7150 3350 50  0001 C CNN
 F 3 "" H 7150 3350 50  0001 C CNN
 F 4 "ACJS-MHOM" H 7050 3500 60  0001 C CNN "mpn"
@@
 $EndComp
 $Comp
-L GND #PWR71
+L GND #PWR047
 U 1 1 5A340D6C
 P 6550 2550
-F 0 "#PWR71" H 6550 2300 50  0001 C CNN
+F 0 "#PWR047" H 6550 2300 50  0001 C CNN
 F 1 "GND" H 6550 2400 50  0000 C CNN
 F 2 "" H 6550 2550 50  0001 C CNN
@@
 Connection ~ 6700 2500
 $Comp
-L GND #PWR72
+L GND #PWR048
 U 1 1 5A340E0A
 P 6600 3850
-F 0 "#PWR72" H 6600 3600 50  0001 C CNN
+F 0 "#PWR048" H 6600 3600 50  0001 C CNN
 F 1 "GND" H 6600 3700 50  0000 C CNN
 F 2 "" H 6600 3850 50  0001 C CNN

Commit message: updated to new kicad format
Parts:
- removed J4, J5: JACK_TRS_6PINS, Connectors:NMJ6HCD2, symbol JACK_TRS_6PINS
- added J4, J5: Audio-Jack-3_3Switches, Connectors:NMJ6HCD2, symbol Connector_Specialized:Audio-Jack-3_3Switches
- C63, C64, C65, C66: symbol C_Small -> Device:C_Small
- U17, U18: symbol DRV135 -> dacparts:DRV135
Connections:
- wire segments 39 -> 47
Changed lines of the file:
@@
-EESchema Schematic File Version 2
-LIBS:power
-LIBS:device
-LIBS:transistors
-LIBS:conn
-LIBS:linear
-LIBS:regul
-LIBS:74xx
-LIBS:cmos4000
-LIBS:adc-dac
-LIBS:memory
-LIBS:xilinx
-LIBS:microcontrollers
-LIBS:dsp
-LIBS:microchip
-LIBS:analog_switches
-LIBS:motorola
-LIBS:texas
-LIBS:intel
-LIBS:audio
-LIBS:interface
-LIBS:digital-audio
-LIBS:philips
-LIBS:display
-LIBS:cypress
-LIBS:siliconi
-LIBS:opto
-LIBS:atmel
-LIBS:contrib
-LIBS:valves
-LIBS:dacparts
-LIBS:USB-DAC-cache
-EELAYER 25 0
+EESchema Schematic File Version 4
+EELAYER 26 0
 EELAYER END
 $Descr A4 11693 8268
 encoding utf-8
-Sheet 5 6
+Sheet 4 6
 Title ""
 Date ""
@@
 $EndDescr
 $Comp
-L DRV135 U17
+L dacparts:DRV135 U17
 U 1 1 5A0DE5A6
 P 5500 2250
@@
 $EndComp
 $Comp
-L C_Small C63
+L Device:C_Small C63
 U 1 1 5A0DE762
 P 4750 2000
@@
 $EndComp
 $Comp
-L C_Small C64
+L Device:C_Small C64
 U 1 1 5A0DE81E
 P 4750 2400
@@
 $EndComp
 Wire Wire Line
-	5000 2400 5000 2550
+	5000 2400 5000 2500
 Wire Wire Line
 	5000 2500 4750 2500
 Wire Wire Line
-	4450 2300 5000 2300
+	4450 2300 4750 2300
 Wire Wire Line
 	4750 1900 5000 1900
 Wire Wire Line
-	5000 1850 5000 2100
+	5000 1850 5000 1900
 Wire Wire Line
 	4750 2100 4750 2300
@@
 	5950 2300 5950 2400
 $Comp
-L GND #PWR041
+L power:GND #PWR041
 U 1 1 5A0DE91C
 P 4450 2350
@@
 Connection ~ 4750 2300
 $Comp
-L +15V #PWR042
+L power:+15V #PWR042
 U 1 1 5A0DE955
 P 5000 1850
@@
 $EndComp
 $Comp
-L -12VA #PWR043
+L power:-12VA #PWR043
 U 1 1 5A0DE975
 P 5000 2550
@@
 	5950 2100 6350 2100
 $Comp
-L DRV135 U18
+L dacparts:DRV135 U18
 U 1 1 5A0DEC40
 P 5500 3450
@@
 $EndComp
 $Comp
-L C_Small C65
+L Device:C_Small C65
 U 1 1 5A0DEC4C
 P 4750 3200
@@
 $EndComp
 $Comp
-L C_Small C66
+L Device:C_Small C66
 U 1 1 5A0DEC52
 P 4750 3600
@@
 $EndComp
 Wire Wire Line
-	5000 3600 5000 3750
+	5000 3600 5000 3700
 Wire Wire Line
 	5000 3700 4750 3700
 Wire Wire Line
-	4450 3500 5000 3500
+	4450 3500 4750 3500
 Wire Wire Line
 	4750 3100 5000 3100
 Wire Wire Line
-	5000 3050 5000 3300
+	5000 3050 5000 3100
 Wire Wire Line
 	4750 3300 4750 3500
@@
 	5950 3500 5950 3600
 $Comp
-L GND #PWR044
+L power:GND #PWR044
 U 1 1 5A0DEC62
 P 4450 3550
@@
 Connection ~ 4750 3500
 $Comp
-L +15V #PWR045
+L power:+15V #PWR045
 U 1 1 5A0DEC6A
 P 5000 3050
@@
 $EndComp
 $Comp
-L -12VA #PWR046
+L power:-12VA #PWR046
 U 1 1 5A0DEC70
 P 5000 3750
@@
 	5950 3300 6150 3300
 $Comp
-L JACK_TRS_6PINS J5
-U 1 1 5A340C41
-P 7150 2300
-AR Path="/5A0DCEAA/5A340C41" Ref="J5"  Part="1"
-AR Path="/59E908E3/5A340C41" Ref="J5"  Part="1"
-F 0 "J5" H 7150 2700 50  0000 C CNN
-F 1 "JACK_TRS_6PINS" H 7100 2000 50  0000 C CNN
-F 2 "Connectors:NMJ6HCD2" H 7250 2150 50  0001 C CNN
-F 3 "" H 7250 2150 50  0001 C CNN
-F 4 "ACJS-MHOM" H 7150 2300 60  0001 C CNN "mpn"
-	1    7150 2300
-	-1   0    0    1
-$EndComp
-$Comp
-L JACK_TRS_6PINS J4
-U 1 1 5A340CC5
-P 7050 3500
-F 0 "J4" H 7050 3900 50  0000 C CNN
-F 1 "JACK_TRS_6PINS" H 7000 3200 50  0000 C CNN
-F 2 "Connectors:NMJ6HCD2" H 7150 3350 50  0001 C CNN
-F 3 "" H 7150 3350 50  0001 C CNN
-F 4 "ACJS-MHOM" H 7050 3500 60  0001 C CNN "mpn"
-	1    7050 3500
-	-1   0    0    1
-$EndComp
-$Comp
-L GND #PWR047
+L power:GND #PWR047
 U 1 1 5A340D6C
 P 6550 2550
@@
 	6550 2550 6550 2500
 Wire Wire Line
-	6550 2500 6750 2500
+	6550 2500 6700 2500
 Wire Wire Line
 	6750 2600 6700 2600
@@
 Connection ~ 6700 2500
 $Comp
-L GND #PWR048
+L power:GND #PWR048
 U 1 1 5A340E0A
 P 6600 3850
@@
 $EndComp
 Wire Wire Line
-	6600 3850 6600 3700
+	6600 3850 6600 3800
 Wire Wire Line
 	6600 3700 6650 3700
@@
 Wire Wire Line
 	6550 2100 6750 2100
+Wire Wire Line
+	4750 2300 5000 2300
+Wire Wire Line
+	5000 2500 5000 2550
+Wire Wire Line
+	5000 1900 5000 2100
+Wire Wire Line
+	4750 3500 5000 3500
+Wire Wire Line
+	5000 3700 5000 3750
+Wire Wire Line
+	5000 3100 5000 3300
+Wire Wire Line
+	6700 2500 6750 2500
+Wire Wire Line
+	6600 3800 6600 3700
+$Comp
+L Connector_Specialized:Audio-Jack-3_3Switches J5
+U 1 1 5A80B063
+P 6950 2400
+F 0 "J5" H 6717 2320 50  0000 R CNN
+F 1 "Audio-Jack-3_3Switches" H 6717 2411 50  0000 R CNN
+F 2 "Connectors:NMJ6HCD2" H 7200 2500 50  0001 C CNN
+F 3 "~" H 7200 2500 50  0001 C CNN
+	1    6950 2400
+	-1   0    0    1
+$EndComp
+$Comp
+L Connector_Specialized:Audio-Jack-3_3Switches J4
+U 1 1 5A80B1AF
+P 6850 3600
+F 0 "J4" H 6617 3520 50  0000 R CNN
+F 1 "Audio-Jack-3_3Switches" H 6617 3611 50  0000 R CNN
+F 2 "Connectors:NMJ6HCD2" H 7100 3700 50  0001 C CNN
+F 3 "~" H 7100 3700 50  0001 C CNN
+	1    6850 3600
+	-1   0    0    1
+$EndComp
 $EndSCHEMATC

Commit message: started routing PCB
Parts:
- C63, C64, C65, C66: footprint Capacitors_SMD:C_0805_HandSoldering -> Capacitors_SMD:C_0402
Connections:
- net labels added: +12V, -12V
- net labels removed: +15V, -12VA
- wire segments 47 -> 51
- no-connect marks 0 -> 4
Changed lines of the file:
@@
 EESchema Schematic File Version 4
+LIBS:USB-DAC-cache
 EELAYER 26 0
 EELAYER END
@@
 F 0 "C63" H 4760 2070 50  0000 L CNN
 F 1 "100n" H 4760 1920 50  0000 L CNN
-F 2 "Capacitors_SMD:C_0805_HandSoldering" H 4750 2000 50  0001 C CNN
+F 2 "Capacitors_SMD:C_0402" H 4750 2000 50  0001 C CNN
 F 3 "" H 4750 2000 50  0001 C CNN
 	1    4750 2000
@@
 F 0 "C64" H 4760 2470 50  0000 L CNN
 F 1 "100n" H 4760 2320 50  0000 L CNN
-F 2 "Capacitors_SMD:C_0805_HandSoldering" H 4750 2400 50  0001 C CNN
+F 2 "Capacitors_SMD:C_0402" H 4750 2400 50  0001 C CNN
 F 3 "" H 4750 2400 50  0001 C CNN
 	1    4750 2400
@@
 	4450 2350 4450 2300
 Connection ~ 4750 2300
-$Comp
-L power:+15V #PWR042
-U 1 1 5A0DE955
-P 5000 1850
-F 0 "#PWR042" H 5000 1700 50  0001 C CNN
-F 1 "+15V" H 5000 1990 50  0000 C CNN
-F 2 "" H 5000 1850 50  0001 C CNN
-F 3 "" H 5000 1850 50  0001 C CNN
-	1    5000 1850
-	1    0    0    -1
-$EndComp
-$Comp
-L power:-12VA #PWR043
-U 1 1 5A0DE975
-P 5000 2550
-F 0 "#PWR043" H 5000 2400 50  0001 C CNN
-F 1 "-12VA" H 5000 2690 50  0000 C CNN
-F 2 "" H 5000 2550 50  0001 C CNN
-F 3 "" H 5000 2550 50  0001 C CNN
-	1    5000 2550
-	-1   0    0    1
-$EndComp
 Connection ~ 5000 2500
 Connection ~ 5000 1900
@@
 F 0 "C65" H 4760 3270 50  0000 L CNN
 F 1 "100n" H 4760 3120 50  0000 L CNN
-F 2 "Capacitors_SMD:C_0805_HandSoldering" H 4750 3200 50  0001 C CNN
+F 2 "Capacitors_SMD:C_0402" H 4750 3200 50  0001 C CNN
 F 3 "" H 4750 3200 50  0001 C CNN
 	1    4750 3200
@@
 F 0 "C66" H 4760 3670 50  0000 L CNN
 F 1 "100n" H 4760 3520 50  0000 L CNN
-F 2 "Capacitors_SMD:C_0805_HandSoldering" H 4750 3600 50  0001 C CNN
+F 2 "Capacitors_SMD:C_0402" H 4750 3600 50  0001 C CNN
 F 3 "" H 4750 3600 50  0001 C CNN
 	1    4750 3600
@@
 Wire Wire Line
 	4950 3400 5000 3400
-Wire Wire Line
-	5950 3400 5950 3300
-Wire Wire Line
-	5950 3500 5950 3600
 $Comp
 L power:GND #PWR044
@@
 	4450 3550 4450 3500
 Connection ~ 4750 3500
-$Comp
-L power:+15V #PWR045
-U 1 1 5A0DEC6A
-P 5000 3050
-F 0 "#PWR045" H 5000 2900 50  0001 C CNN
-F 1 "+15V" H 5000 3190 50  0000 C CNN
-F 2 "" H 5000 3050 50  0001 C CNN
-F 3 "" H 5000 3050 50  0001 C CNN
-	1    5000 3050
-	1    0    0    -1
-$EndComp
-$Comp
-L power:-12VA #PWR046
-U 1 1 5A0DEC70
-P 5000 3750
-F 0 "#PWR046" H 5000 3600 50  0001 C CNN
-F 1 "-12VA" H 5000 3890 50  0000 C CNN
-F 2 "" H 5000 3750 50  0001 C CNN
-F 3 "" H 5000 3750 50  0001 C CNN
-	1    5000 3750
-	-1   0    0    1
-$EndComp
 Connection ~ 5000 3700
 Connection ~ 5000 3100
 Wire Wire Line
-	5950 3600 6400 3600
-Wire Wire Line
-	5950 3300 6150 3300
+	5950 3600 6000 3600
+Wire Wire Line
+	5950 3300 6000 3300
 $Comp
 L power:GND #PWR047
@@
 	-1   0    0    1
 $EndComp
+$Comp
+L power:+12V #PWR035
+U 1 1 5A7D6CAB
+P 5000 1850
+F 0 "#PWR035" H 5000 1700 50  0001 C CNN
+F 1 "+12V" H 5015 2023 50  0000 C CNN
+F 2 "" H 5000 1850 50  0001 C CNN
+F 3 "" H 5000 1850 50  0001 C CNN
+	1    5000 1850
+	1    0    0    -1
+$EndComp
+$Comp
+L power:-12V #PWR46
+U 1 1 5A7D6D39
+P 5000 3750
+F 0 "#PWR46" H 5000 3850 50  0001 C CNN
+F 1 "-12V" H 5015 3923 50  0000 C CNN
+F 2 "" H 5000 3750 50  0001 C CNN
+F 3 "" H 5000 3750 50  0001 C CNN
+	1    5000 3750
+	-1   0    0    1
+$EndComp
+$Comp
+L power:+12V #PWR036
+U 1 1 5A7D6EBF
+P 5000 3050
+F 0 "#PWR036" H 5000 2900 50  0001 C CNN
+F 1 "+12V" H 5015 3223 50  0000 C CNN
+F 2 "" H 5000 3050 50  0001 C CNN
+F 3 "" H 5000 3050 50  0001 C CNN
+	1    5000 3050
+	1    0    0    -1
+$EndComp
+$Comp
+L power:-12V #PWR45
+U 1 1 5A7D7AAD
+P 5000 2550
+F 0 "#PWR45" H 5000 2650 50  0001 C CNN
+F 1 "-12V" H 5015 2723 50  0000 C CNN
+F 2 "" H 5000 2550 50  0001 C CNN
+F 3 "" H 5000 2550 50  0001 C CNN
+	1    5000 2550
+	-1   0    0    1
+$EndComp
+Wire Wire Line
+	5950 3400 6000 3400
+Wire Wire Line
+	6000 3400 6000 3300
+Connection ~ 6000 3300
+Wire Wire Line
+	6000 3300 6150 3300
+Wire Wire Line
+	5950 3500 6000 3500
+Wire Wire Line
+	6000 3500 6000 3600
+Connection ~ 6000 3600
+Wire Wire Line
+	6000 3600 6400 3600
+NoConn ~ 6650 3600
+NoConn ~ 6650 3400
+NoConn ~ 6750 2200
+NoConn ~ 6750 2400
 $EndSCHEMATC
