File: file5A0DFAF0.sch (KiCad schematic (older format))
At the start: 10 parts, among them J6 JACK_TRS_6PINS, U19 TPA6120A2

Commit message: Updated schematics and part number fields
Parts:
- R34: value 50 -> 51; MPN (none) -> RC0805FR-0751RL
- R40: MPN (none) -> RC0805FR-0739R2L
- U19: footprint (none) -> Housings_SOIC:SOIC-20W_7.5x12.8mm_Pitch1.27mm
Changed lines of the file:
@@
 F 0 "U19" H 4300 2650 60  0000 C CNN
 F 1 "TPA6120A2" H 4400 2350 60  0000 C CNN
-F 2 "" H 4050 2500 60  0001 C CNN
+F 2 "Housings_SOIC:SOIC-20W_7.5x12.8mm_Pitch1.27mm" H 4050 2500 60  0001 C CNN
 F 3 "" H 4050 2500 60  0001 C CNN
 F 4 "TPA6120A2DWPR" H 4050 2500 60  0001 C CNN "mpn"
@@
 F 0 "U19" H 4300 3950 60  0000 C CNN
 F 1 "TPA6120A2" H 4400 3650 60  0000 C CNN
-F 2 "" H 4050 3800 60  0001 C CNN
+F 2 "Housings_SOIC:SOIC-20W_7.5x12.8mm_Pitch1.27mm" H 4050 3800 60  0001 C CNN
 F 3 "" H 4050 3800 60  0001 C CNN
 	2    4050 3800
@@
 $EndComp
 $Comp
-L +15V #PWR073
+L +15V #PWR75
 U 1 1 5A0EF3B4
 P 4050 2150
-F 0 "#PWR073" H 4050 2000 50  0001 C CNN
+F 0 "#PWR75" H 4050 2000 50  0001 C CNN
 F 1 "+15V" H 4050 2290 50  0000 C CNN
 F 2 "" H 4050 2150 50  0001 C CNN
@@
 	4050 2150 4050 2200
 $Comp
-L -12VA #PWR074
+L -12VA #PWR76
 U 1 1 5A0EF3DD
 P 4050 2850
-F 0 "#PWR074" H 4050 2700 50  0001 C CNN
+F 0 "#PWR76" H 4050 2700 50  0001 C CNN
 F 1 "-12VA" H 4050 2990 50  0000 C CNN
 F 2 "" H 4050 2850 50  0001 C CNN
@@
 $EndComp
 $Comp
-L GND #PWR075
+L GND #PWR73
 U 1 1 5A0EF50D
 P 3350 2600
-F 0 "#PWR075" H 3350 2350 50  0001 C CNN
+F 0 "#PWR73" H 3350 2350 50  0001 C CNN
 F 1 "GND" H 3350 2450 50  0000 C CNN
 F 2 "" H 3350 2600 50  0001 C CNN
@@
 P 3600 2400
 F 0 "R34" V 3680 2400 50  0000 C CNN
-F 1 "50" V 3600 2400 50  0000 C CNN
+F 1 "51" V 3600 2400 50  0000 C CNN
 F 2 "Resistors_SMD:R_0805_HandSoldering" V 3530 2400 50  0001 C CNN
 F 3 "" H 3600 2400 50  0001 C CNN
+F 4 "RC0805FR-0751RL" V 3600 2400 60  0001 C CNN "MPN"
 	1    3600 2400
 	0    -1   -1   0
@@
 F 2 "Resistors_SMD:R_0805_HandSoldering" V 4530 2500 50  0001 C CNN
 F 3 "" H 4600 2500 50  0001 C CNN
+F 4 "RC0805FR-0739R2L" V 4600 2500 60  0001 C CNN "MPN"
 	1    4600 2500
 	0    -1   -1   0
@@
 	3750 2400 3800 2400
 $Comp
-L +15V #PWR076
+L +15V #PWR77
 U 1 1 5A0EF892
 P 4050 3450
-F 0 "#PWR076" H 4050 3300 50  0001 C CNN
+F 0 "#PWR77" H 4050 3300 50  0001 C CNN
 F 1 "+15V" H 4050 3590 50  0000 C CNN
 F 2 "" H 4050 3450 50  0001 C CNN
@@
 	4050 3450 4050 3500
 $Comp
-L -12VA #PWR077
+L -12VA #PWR78
 U 1 1 5A0EF899
 P 4050 4150
-F 0 "#PWR077" H 4050 4000 50  0001 C CNN
+F 0 "#PWR78" H 4050 4000 50  0001 C CNN
 F 1 "-12VA" H 4050 4290 50  0000 C CNN
 F 2 "" H 4050 4150 50  0001 C CNN
@@
 $EndComp
 $Comp
-L GND #PWR078
+L GND #PWR74
 U 1 1 5A0EF8A6
 P 3350 3900
-F 0 "#PWR078" H 3350 3650 50  0001 C CNN
+F 0 "#PWR74" H 3350 3650 50  0001 C CNN
 F 1 "GND" H 3350 3750 50  0000 C CNN
 F 2 "" H 3350 3900 50  0001 C CNN
@@
 	3750 3700 3800 3700
 $Comp
-L GND #PWR079
+L GND #PWR79
 U 1 1 5A0EF9D3
 P 5050 3300
-F 0 "#PWR079" H 5050 3050 50  0001 C CNN
+F 0 "#PWR79" H 5050 3050 50  0001 C CNN
 F 1 "GND" H 5050 3150 50  0000 C CNN
 F 2 "" H 5050 3300 50  0001 C CNN

Commit message: Began PCB layout
Parts:
- J6: footprint (none) -> Connectors:NMJ6HCD2
- R36: value 50 -> 51
Changed lines of the file:
@@
 $EndComp
 $Comp
-L +15V #PWR75
+L +15V #PWR049
 U 1 1 5A0EF3B4
 P 4050 2150
-F 0 "#PWR75" H 4050 2000 50  0001 C CNN
+F 0 "#PWR049" H 4050 2000 50  0001 C CNN
 F 1 "+15V" H 4050 2290 50  0000 C CNN
 F 2 "" H 4050 2150 50  0001 C CNN
@@
 	4050 2150 4050 2200
 $Comp
-L -12VA #PWR76
+L -12VA #PWR050
 U 1 1 5A0EF3DD
 P 4050 2850
-F 0 "#PWR76" H 4050 2700 50  0001 C CNN
+F 0 "#PWR050" H 4050 2700 50  0001 C CNN
 F 1 "-12VA" H 4050 2990 50  0000 C CNN
 F 2 "" H 4050 2850 50  0001 C CNN
@@
 $EndComp
 $Comp
-L GND #PWR73
+L GND #PWR051
 U 1 1 5A0EF50D
 P 3350 2600
-F 0 "#PWR73" H 3350 2350 50  0001 C CNN
+F 0 "#PWR051" H 3350 2350 50  0001 C CNN
 F 1 "GND" H 3350 2450 50  0000 C CNN
 F 2 "" H 3350 2600 50  0001 C CNN
@@
 	3750 2400 3800 2400
 $Comp
-L +15V #PWR77
+L +15V #PWR052
 U 1 1 5A0EF892
 P 4050 3450
-F 0 "#PWR77" H 4050 3300 50  0001 C CNN
+F 0 "#PWR052" H 4050 3300 50  0001 C CNN
 F 1 "+15V" H 4050 3590 50  0000 C CNN
 F 2 "" H 4050 3450 50  0001 C CNN
@@
 	4050 3450 4050 3500
 $Comp
-L -12VA #PWR78
+L -12VA #PWR053
 U 1 1 5A0EF899
 P 4050 4150
-F 0 "#PWR78" H 4050 4000 50  0001 C CNN
+F 0 "#PWR053" H 4050 4000 50  0001 C CNN
 F 1 "-12VA" H 4050 4290 50  0000 C CNN
 F 2 "" H 4050 4150 50  0001 C CNN
@@
 $EndComp
 $Comp
-L GND #PWR74
+L GND #PWR054
 U 1 1 5A0EF8A6
 P 3350 3900
-F 0 "#PWR74" H 3350 3650 50  0001 C CNN
+F 0 "#PWR054" H 3350 3650 50  0001 C CNN
 F 1 "GND" H 3350 3750 50  0000 C CNN
 F 2 "" H 3350 3900 50  0001 C CNN
@@
 P 3600 3700
 F 0 "R36" V 3680 3700 50  0000 C CNN
-F 1 "50" V 3600 3700 50  0000 C CNN
+F 1 "51" V 3600 3700 50  0000 C CNN
 F 2 "Resistors_SMD:R_0805_HandSoldering" V 3530 3700 50  0001 C CNN
 F 3 "" H 3600 3700 50  0001 C CNN
@@
 	3750 3700 3800 3700
 $Comp
-L GND #PWR79
+L GND #PWR055
 U 1 1 5A0EF9D3
 P 5050 3300
-F 0 "#PWR79" H 5050 3050 50  0001 C CNN
+F 0 "#PWR055" H 5050 3050 50  0001 C CNN
 F 1 "GND" H 5050 3150 50  0000 C CNN
 F 2 "" H 5050 3300 50  0001 C CNN
@@
 F 0 "J6" H 5600 3650 50  0000 C CNN
 F 1 "JACK_TRS_6PINS" H 5550 2950 50  0000 C CNN
-F 2 "" H 5700 3100 50  0001 C CNN
+F 2 "Connectors:NMJ6HCD2" H 5700 3100 50  0001 C CNN
 F 3 "" H 5700 3100 50  0001 C CNN
 	1    5600 3250

Commit message: updated to new kicad format
Parts:
- removed J6: JACK_TRS_6PINS, Connectors:NMJ6HCD2, symbol JACK_TRS_6PINS
- added J6: Audio-Jack-3_3Switches, Connectors:NMJ6HCD2, symbol Connector_Specialized:Audio-Jack-3_3Switches
- R34, R35, R36, R37, R38, R39, R40, R41: symbol R -> Device:R
- U19: symbol TPA6120A2 -> dacparts:TPA6120A2
Connections:
- wire segments 28 -> 29
Changed lines of the file:
@@
-EESchema Schematic File Version 2
-LIBS:power
-LIBS:device
-LIBS:transistors
-LIBS:conn
-LIBS:linear
-LIBS:regul
-LIBS:74xx
-LIBS:cmos4000
-LIBS:adc-dac
-LIBS:memory
-LIBS:xilinx
-LIBS:microcontrollers
-LIBS:dsp
-LIBS:microchip
-LIBS:analog_switches
-LIBS:motorola
-LIBS:texas
-LIBS:intel
-LIBS:audio
-LIBS:interface
-LIBS:digital-audio
-LIBS:philips
-LIBS:display
-LIBS:cypress
-LIBS:siliconi
-LIBS:opto
-LIBS:atmel
-LIBS:contrib
-LIBS:valves
-LIBS:dacparts
-LIBS:USB-DAC-cache
-EELAYER 25 0
+EESchema Schematic File Version 4
+EELAYER 26 0
 EELAYER END
 $Descr A4 11693 8268
 encoding utf-8
-Sheet 6 6
+Sheet 5 6
 Title ""
 Date ""
@@
 $EndDescr
 $Comp
-L TPA6120A2 U19
+L dacparts:TPA6120A2 U19
 U 1 1 5A0EF2B2
 P 4050 2500
@@
 $EndComp
 $Comp
-L TPA6120A2 U19
+L dacparts:TPA6120A2 U19
 U 2 1 5A0EF325
 P 4050 3800
@@
 $EndComp
 $Comp
-L +15V #PWR049
+L power:+15V #PWR049
 U 1 1 5A0EF3B4
 P 4050 2150
@@
 	4050 2150 4050 2200
 $Comp
-L -12VA #PWR050
+L power:-12VA #PWR050
 U 1 1 5A0EF3DD
 P 4050 2850
@@
 	4050 2850 4050 2800
 $Comp
-L R R35
+L Device:R R35
 U 1 1 5A0EF3FA
 P 3600 2600
@@
 $EndComp
 $Comp
-L GND #PWR051
+L power:GND #PWR051
 U 1 1 5A0EF50D
 P 3350 2600
@@
 	3750 2600 3800 2600
 $Comp
-L R R38
+L Device:R R38
 U 1 1 5A0EF537
 P 4050 3150
@@
 	4400 3150 4400 2500
 $Comp
-L R R34
+L Device:R R34
 U 1 1 5A0EF58F
 P 3600 2400
@@
 $EndComp
 $Comp
-L R R40
+L Device:R R40
 U 1 1 5A0EF5D1
 P 4600 2500
@@
 	3750 2400 3800 2400
 $Comp
-L +15V #PWR052
+L power:+15V #PWR052
 U 1 1 5A0EF892
 P 4050 3450
@@
 	4050 3450 4050 3500
 $Comp
-L -12VA #PWR053
+L power:-12VA #PWR053
 U 1 1 5A0EF899
 P 4050 4150
@@
 	4050 4150 4050 4100
 $Comp
-L R R37
+L Device:R R37
 U 1 1 5A0EF8A0
 P 3600 3900
@@
 $EndComp
 $Comp
-L GND #PWR054
+L power:GND #PWR054
 U 1 1 5A0EF8A6
 P 3350 3900
@@
 	3750 3900 3800 3900
 $Comp
-L R R39
+L Device:R R39
 U 1 1 5A0EF8AE
 P 4050 4450
@@
 	4400 4450 4400 3800
 $Comp
-L R R36
+L Device:R R36
 U 1 1 5A0EF8B8
 P 3600 3700
@@
 $EndComp
 $Comp
-L R R41
+L Device:R R41
 U 1 1 5A0EF8BE
 P 4600 3800
@@
 	3750 3700 3800 3700
 $Comp
-L GND #PWR055
+L power:GND #PWR055
 U 1 1 5A0EF9D3
 P 5050 3300
@@
 Wire Wire Line
 	5200 2500 5200 3050
-$Comp
-L JACK_TRS_6PINS J6
-U 1 1 5A0EF6A5
-P 5600 3250
-F 0 "J6" H 5600 3650 50  0000 C CNN
-F 1 "JACK_TRS_6PINS" H 5550 2950 50  0000 C CNN
-F 2 "Connectors:NMJ6HCD2" H 5700 3100 50  0001 C CNN
-F 3 "" H 5700 3100 50  0001 C CNN
-	1    5600 3250
-	-1   0    0    1
-$EndComp
 Wire Wire Line
 	5050 3300 5200 3300
 Wire Wire Line
-	5200 3250 5200 3350
+	5200 3250 5200 3300
 Connection ~ 5200 3300
 Wire Wire Line
@@
 NoConn ~ 5200 3150
 NoConn ~ 5200 3550
+Wire Wire Line
+	5200 3300 5200 3350
+$Comp
+L Connector_Specialized:Audio-Jack-3_3Switches J6
+U 1 1 5A784233
+P 5800 3250
+F 0 "J6" H 5804 3675 50  0000 C CNN
+F 1 "Audio-Jack-3_3Switches" H 5804 3584 50  0000 C CNN
+F 2 "Connectors:NMJ6HCD2" H 6050 3350 50  0001 C CNN
+F 3 "~" H 6050 3350 50  0001 C CNN
+	1    5800 3250
+	-1   0    0    -1
+$EndComp
 $EndSCHEMATC

Commit message: started routing PCB
Parts:
- R34, R36, R40, R41: footprint Resistors_SMD:R_0805_HandSoldering -> Resistors_SMD:R_0805
- R35, R37, R38, R39: footprint Resistors_SMD:R_0805_HandSoldering -> Resistors_SMD:R_0402
Connections:
- net labels added: +12V, -12V
- net labels removed: +15V, -12VA
Changed lines of the file:
@@
 EESchema Schematic File Version 4
+LIBS:USB-DAC-cache
 EELAYER 26 0
 EELAYER END
@@
 	1    0    0    -1
 $EndComp
-$Comp
-L power:+15V #PWR049
-U 1 1 5A0EF3B4
-P 4050 2150
-F 0 "#PWR049" H 4050 2000 50  0001 C CNN
-F 1 "+15V" H 4050 2290 50  0000 C CNN
-F 2 "" H 4050 2150 50  0001 C CNN
-F 3 "" H 4050 2150 50  0001 C CNN
-	1    4050 2150
-	1    0    0    -1
-$EndComp
 Wire Wire Line
 	4050 2150 4050 2200
-$Comp
-L power:-12VA #PWR050
-U 1 1 5A0EF3DD
-P 4050 2850
-F 0 "#PWR050" H 4050 2700 50  0001 C CNN
-F 1 "-12VA" H 4050 2990 50  0000 C CNN
-F 2 "" H 4050 2850 50  0001 C CNN
-F 3 "" H 4050 2850 50  0001 C CNN
-	1    4050 2850
-	-1   0    0    1
-$EndComp
 Wire Wire Line
 	4050 2850 4050 2800
@@
 F 0 "R35" V 3680 2600 50  0000 C CNN
 F 1 "1K" V 3600 2600 50  0000 C CNN
-F 2 "Resistors_SMD:R_0805_HandSoldering" V 3530 2600 50  0001 C CNN
+F 2 "Resistors_SMD:R_0402" V 3530 2600 50  0001 C CNN
 F 3 "" H 3600 2600 50  0001 C CNN
 	1    3600 2600
@@
 F 0 "R38" V 4130 3150 50  0000 C CNN
 F 1 "1K" V 4050 3150 50  0000 C CNN
-F 2 "Resistors_SMD:R_0805_HandSoldering" V 3980 3150 50  0001 C CNN
+F 2 "Resistors_SMD:R_0402" V 3980 3150 50  0001 C CNN
 F 3 "" H 4050 3150 50  0001 C CNN
 	1    4050 3150
@@
 F 0 "R34" V 3680 2400 50  0000 C CNN
 F 1 "51" V 3600 2400 50  0000 C CNN
-F 2 "Resistors_SMD:R_0805_HandSoldering" V 3530 2400 50  0001 C CNN
+F 2 "Resistors_SMD:R_0805" V 3530 2400 50  0001 C CNN
 F 3 "" H 3600 2400 50  0001 C CNN
 F 4 "RC0805FR-0751RL" V 3600 2400 60  0001 C CNN "MPN"
@@
 F 0 "R40" V 4680 2500 50  0000 C CNN
 F 1 "39.2" V 4600 2500 50  0000 C CNN
-F 2 "Resistors_SMD:R_0805_HandSoldering" V 4530 2500 50  0001 C CNN
+F 2 "Resistors_SMD:R_0805" V 4530 2500 50  0001 C CNN
 F 3 "" H 4600 2500 50  0001 C CNN
 F 4 "RC0805FR-0739R2L" V 4600 2500 60  0001 C CNN "MPN"
@@
 Wire Wire Line
 	3750 2400 3800 2400
-$Comp
-L power:+15V #PWR052
-U 1 1 5A0EF892
-P 4050 3450
-F 0 "#PWR052" H 4050 3300 50  0001 C CNN
-F 1 "+15V" H 4050 3590 50  0000 C CNN
-F 2 "" H 4050 3450 50  0001 C CNN
-F 3 "" H 4050 3450 50  0001 C CNN
-	1    4050 3450
-	1    0    0    -1
-$EndComp
 Wire Wire Line
 	4050 3450 4050 3500
-$Comp
-L power:-12VA #PWR053
-U 1 1 5A0EF899
-P 4050 4150
-F 0 "#PWR053" H 4050 4000 50  0001 C CNN
-F 1 "-12VA" H 4050 4290 50  0000 C CNN
-F 2 "" H 4050 4150 50  0001 C CNN
-F 3 "" H 4050 4150 50  0001 C CNN
-	1    4050 4150
-	-1   0    0    1
-$EndComp
 Wire Wire Line
 	4050 4150 4050 4100
@@
 F 0 "R37" V 3680 3900 50  0000 C CNN
 F 1 "1K" V 3600 3900 50  0000 C CNN
-F 2 "Resistors_SMD:R_0805_HandSoldering" V 3530 3900 50  0001 C CNN
+F 2 "Resistors_SMD:R_0402" V 3530 3900 50  0001 C CNN
 F 3 "" H 3600 3900 50  0001 C CNN
 	1    3600 3900
@@
 F 0 "R39" V 4130 4450 50  0000 C CNN
 F 1 "1K" V 4050 4450 50  0000 C CNN
-F 2 "Resistors_SMD:R_0805_HandSoldering" V 3980 4450 50  0001 C CNN
+F 2 "Resistors_SMD:R_0402" V 3980 4450 50  0001 C CNN
 F 3 "" H 4050 4450 50  0001 C CNN
 	1    4050 4450
@@
 F 0 "R36" V 3680 3700 50  0000 C CNN
 F 1 "51" V 3600 3700 50  0000 C CNN
-F 2 "Resistors_SMD:R_0805_HandSoldering" V 3530 3700 50  0001 C CNN
+F 2 "Resistors_SMD:R_0805" V 3530 3700 50  0001 C CNN
 F 3 "" H 3600 3700 50  0001 C CNN
 	1    3600 3700
@@
 F 0 "R41" V 4680 3800 50  0000 C CNN
 F 1 "39.2" V 4600 3800 50  0000 C CNN
-F 2 "Resistors_SMD:R_0805_HandSoldering" V 4530 3800 50  0001 C CNN
+F 2 "Resistors_SMD:R_0805" V 4530 3800 50  0001 C CNN
 F 3 "" H 4600 3800 50  0001 C CNN
 	1    4600 3800
@@
 L Connector_Specialized:Audio-Jack-3_3Switches J6
 U 1 1 5A784233
-P 5800 3250
-F 0 "J6" H 5804 3675 50  0000 C CNN
-F 1 "Audio-Jack-3_3Switches" H 5804 3584 50  0000 C CNN
-F 2 "Connectors:NMJ6HCD2" H 6050 3350 50  0001 C CNN
-F 3 "~" H 6050 3350 50  0001 C CNN
-	1    5800 3250
+P 5400 3250
+F 0 "J6" H 5404 3675 50  0000 C CNN
+F 1 "Audio-Jack-3_3Switches" H 5404 3584 50  0000 C CNN
+F 2 "Connectors:NMJ6HCD2" H 5650 3350 50  0001 C CNN
+F 3 "~" H 5650 3350 50  0001 C CNN
+	1    5400 3250
 	-1   0    0    -1
 $EndComp
+$Comp
+L power:+12V #PWR042
+U 1 1 5A7D769F
+P 4050 2150
+F 0 "#PWR042" H 4050 2000 50  0001 C CNN
+F 1 "+12V" H 4065 2323 50  0000 C CNN
+F 2 "" H 4050 2150 50  0001 C CNN
+F 3 "" H 4050 2150 50  0001 C CNN
+	1    4050 2150
+	1    0    0    -1
+$EndComp
+$Comp
+L power:-12V #PWR49
+U 1 1 5A7D7BA2
+P 4050 2850
+F 0 "#PWR49" H 4050 2950 50  0001 C CNN
+F 1 "-12V" H 4065 3023 50  0000 C CNN
+F 2 "" H 4050 2850 50  0001 C CNN
+F 3 "" H 4050 2850 50  0001 C CNN
+	1    4050 2850
+	-1   0    0    1
+$EndComp
+$Comp
+L power:+12V #PWR043
+U 1 1 5A7D7C71
+P 4050 3450
+F 0 "#PWR043" H 4050 3300 50  0001 C CNN
+F 1 "+12V" H 4065 3623 50  0000 C CNN
+F 2 "" H 4050 3450 50  0001 C CNN
+F 3 "" H 4050 3450 50  0001 C CNN
+	1    4050 3450
+	1    0    0    -1
+$EndComp
+$Comp
+L power:-12V #PWR50
+U 1 1 5A7D7D2C
+P 4050 4150
+F 0 "#PWR50" H 4050 4250 50  0001 C CNN
+F 1 "-12V" H 4065 4323 50  0000 C CNN
+F 2 "" H 4050 4150 50  0001 C CNN
+F 3 "" H 4050 4150 50  0001 C CNN
+	1    4050 4150
+	-1   0    0    1
+$EndComp
 $EndSCHEMATC
